File: GPIOBoard/CAN.kicad_sch (KiCad schematic)
At the start: 7 parts, among them U4 MCP2561/2FD

Commit message: GPIO Board ver1.1
Parts:
- C12: Name CL10B104KA8NNNC -> GCJ188R91H124KA01D; Price 12 -> 36; URL https://www.digikey.jp/ja/products/detail/samsung-electro-m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 -> https://www.digikey.jp/ja/products/detail/murata-electronic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
- D13, D14: Name SML-E12P8WT86 -> SML-D14MWT86A; Price 39 -> 53; URL https://www.digikey.jp/ja/products/detail/rohm-semiconductor/SML-E12P8WT86/1641804 -> https://www.digikey.jp/ja/products/detail/rohm-semiconductor/SML-D14MWT86A/9448204
- R23, R24: value 55 -> 96; Name ESR03EZPF60R4 -> ESR03EZPJ101; Price 23 -> 22; URL https://www.digikey.jp/ja/products/detail/rohm-semiconductor/ESR03EZPF60R4/20486478 -> https://www.digikey.jp/ja/products/detail/rohm-semiconductor/ESR03EZPJ101/1983452
Other:
- note added: "Vcc = 3.3V Vf = 2.1V, If = 12.5mA (3.3-2.1) / 0.0125 = 96Ω"
- note removed: "Vcc = 3.3V Vf = 2.2V, If = 20mA (3.3-2.2) / 0.02 = 55Ω"
- company: (none) -> 阿南高専ロボット研究部
- title: (none) -> GPIO Board / CAN
Changed lines of the file:
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@@
 	(generator_version "9.0")
 	(paper "A4")
+	(title_block
+		(title "GPIO Board / CAN")
+		(date "2025-04-03")
+		(rev "ver1.1")
+		(company "阿南高専ロボット研究部")
+	)
 	(text "MCP2562FDを使うならジャンパする"
 		(exclude_from_sim no)
@@
 		)
 	)
-	(text "Vcc = 3.3V\nVf = 2.2V, If = 20mA\n\n(3.3-2.2) / 0.02 = 55Ω"
+	(text "Vcc = 3.3V\nVf = 2.1V, If = 12.5mA\n\n(3.3-2.1) / 0.0125 = 96Ω"
 		(exclude_from_sim no)
 		(at 135.636 103.632 0)
@@
 			)
 		)
-		(property "Name" "SML-E12P8WT86"
+		(property "Name" "SML-D14MWT86A"
 			(at 130.81 86.36 0)
 			(effects
@@
 			)
 		)
-		(property "URL" "https://www.digikey.jp/ja/products/detail/rohm-semiconductor/SML-E12P8WT86/1641804"
+		(property "URL" "https://www.digikey.jp/ja/products/detail/rohm-semiconductor/SML-D14MWT86A/9448204"
 			(at 130.81 86.36 0)
 			(effects
@@
 			)
 		)
-		(property "Price" "39"
+		(property "Price" "53"
 			(at 130.81 86.36 0)
 			(effects
@@
 			)
 		)
-		(property "Name" "CL10B104KA8NNNC"
+		(property "Name" "GCJ188R91H124KA01D"
 			(at 151.13 64.77 0)
 			(effects
@@
 			)
 		)
-		(property "URL" "https://www.digikey.jp/ja/products/detail/samsung-electro-mechanics/CL10B104KA8NNNC/3886664"
+		(property "URL" "https://www.digikey.jp/ja/products/detail/murata-electronics/GCJ188R91H124KA01D/13401917"
 			(at 151.13 64.77 0)
 			(effects
@@
 			)
 		)
-		(property "Price" "12"
+		(property "Price" "36"
 			(at 151.13 64.77 0)
 			(effects
@@
 	)
 	(symbol
+		(lib_name "LED_1")
 		(lib_id "Device:LED")
 		(at 124.46 86.36 90)
@@
 			)
 		)
-		(property "Name" "SML-E12P8WT86"
+		(property "Name" "SML-D14MWT86A"
 			(at 124.46 86.36 0)
 			(effects
@@
 			)
 		)
-		(property "URL" "https://www.digikey.jp/ja/products/detail/rohm-semiconductor/SML-E12P8WT86/1641804"
+		(property "URL" "https://www.digikey.jp/ja/products/detail/rohm-semiconductor/SML-D14MWT86A/9448204"
 			(at 124.46 86.36 0)
 			(effects
@@
 			)
 		)
-		(property "Price" "39"
+		(property "Price" "53"
 			(at 124.46 86.36 0)
 			(effects
@@
 			)
 		)
-		(property "Value" "55"
+		(property "Value" "96"
 			(at 122.174 96.52 0)
 			(effects
@@
 			)
 		)
-		(property "Name" "ESR03EZPF60R4"
+		(property "Name" "ESR03EZPJ101"
 			(at 124.46 95.25 0)
 			(effects
@@
 			)
 		)
-		(property "URL" "https://www.digikey.jp/ja/products/detail/rohm-semiconductor/ESR03EZPF60R4/20486478"
+		(property "URL" "https://www.digikey.jp/ja/products/detail/rohm-semiconductor/ESR03EZPJ101/1983452"
 			(at 124.46 95.25 0)
 			(effects
@@
 			)
 		)
-		(property "Price" "23"
+		(property "Price" "22"
 			(at 124.46 95.25 0)
 			(effects
@@
 			)
 		)
-		(property "Value" "55"
+		(property "Value" "96"
 			(at 133.35 96.5199 0)
 			(effects
@@
 			)
 		)
-		(property "Name" "ESR03EZPF60R4"
+		(property "Name" "ESR03EZPJ101"
 			(at 130.81 95.25 0)
 			(effects
@@
 			)
 		)
-		(property "URL" "https://www.digikey.jp/ja/products/detail/rohm-semiconductor/ESR03EZPF60R4/20486478"
+		(property "URL" "https://www.digikey.jp/ja/products/detail/rohm-semiconductor/ESR03EZPJ101/1983452"
 			(at 130.81 95.25 0)
 			(effects
@@
 			)
 		)
-		(property "Price" "23"
+		(property "Price" "22"
 			(at 130.81 95.25 0)
 			(effects
