File: GPIOBoard/MCU.kicad_sch (KiCad schematic)
At the start: 14 parts, among them J11 SWD, SW1 RESET, U1 STM32F303K8Tx, Y1 Crystal_GND2

Commit message: GPIO Board ver1.1
Parts:
- added R31: 10k, Resistor_SMD:R_0603_1608Metric, symbol Device:R
- C10, C9: Name C0603C150K4GACTU -> GCM1885C2A150JA16D; URL https://www.digikey.jp/ja/products/detail/kemet/C0603C150K4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 -> https://www.digikey.jp/ja/products/detail/murata-electronic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
- C3, C4, C6, C8: Name CL10B104KA8NNNC -> GCJ188R91H124KA01D; Price 12 -> 36; URL https://www.digikey.jp/ja/products/detail/samsung-electro-m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 -> https://www.digikey.jp/ja/products/detail/murata-electronic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
- C5: Name CL10A106KQ8NNNC -> GRM188R60G106ME47D; Price 12 -> 19; URL https://www.digikey.jp/ja/products/detail/samsung-electro-m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 -> https://www.digikey.jp/ja/products/detail/murata-electronic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
- C7: Name CL10B105KA8NNNC -> GRM188D71H105ME01W; Price 9 -> 47; URL https://www.digikey.jp/ja/products/detail/samsung-electro-m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 -> https://www.digikey.jp/ja/products/detail/murata-electronic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
- R26: Name ESR03EZPF1002 -> ESR03EZPJ103; Price 23 -> 22; URL https://www.digikey.jp/ja/products/detail/rohm-semiconductor/ESR03EZPF1002/1983429 -> https://www.digikey.jp/ja/products/detail/rohm-semiconductor/ESR03EZPJ103/1762722
Connections:
- net +3.3V: now also R31.1
- net at R26.1, U1.31 (BOOT0): now also R31.2
- net LED_R: now reaches U1.10 (PA4)
- net LED_G: now reaches U1.18 (PA8)
- net LED_B: now reaches U1.6 (PA0)
Other:
- company: (none) -> 阿南高専ロボット研究部
- title: (none) -> GPIO Board / MCU
