File: GPIOBoard/USB-UART.kicad_sch (KiCad schematic)
At the start: 9 parts, among them J10 Debug, U3 CH340E

Commit message: GPIO Board ver1.1
Parts:
- C11: Name CL10B104KA8NNNC -> GCJ188R91H124KA01D; Price 12 -> 36; URL https://www.digikey.jp/ja/products/detail/samsung-electro-m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 -> https://www.digikey.jp/ja/products/detail/murata-electronic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
- D12: value data -> Data; Name SML-E12P8WT86 -> SML-D14MWT86A; Price 39 -> 53; URL https://www.digikey.jp/ja/products/detail/rohm-semiconductor/SML-E12P8WT86/1641804 -> https://www.digikey.jp/ja/products/detail/rohm-semiconductor/SML-D14MWT86A/9448204
- D15: footprint Diode_SMD:D_SOD-123 -> Diode_SMD:Nexperia_CFP3_SOD-123W; Name RB160M-30TR -> PMEG3010ER,115; Price 15 -> 30; URL https://akizukidenshi.com/catalog/g/g101398/ -> https://www.digikey.jp/ja/products/detail/nexperia-usa-inc/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
- R20: value 55 -> 96; Name ESR03EZPF60R4 -> ESR03EZPJ101; Price 23 -> 22; URL https://www.digikey.jp/ja/products/detail/rohm-semiconductor/ESR03EZPF60R4/20486478 -> https://www.digikey.jp/ja/products/detail/rohm-semiconductor/ESR03EZPJ101/1983452
- R21, R22: Name ESR03EZPF5101 -> ESR03EZPJ512; Price 23 -> 22; URL https://www.digikey.jp/ja/products/detail/rohm-semiconductor/ESR03EZPF5101/4007250 -> https://www.digikey.jp/ja/products/detail/rohm-semiconductor/ESR03EZPJ512/1762735
Other:
- note added: "Vcc = 3.3V Vf = 2.1V, If = 12.5mA (3.3-2.1) / 0.0125 = 96Ω"
- note removed: "Vcc = 3.3V Vf = 2.2V, If = 20mA (3.3-2.2) / 0.02 = 55Ω"
- company: (none) -> 阿南高専ロボット研究部
- title: (none) -> GPIO Board / USB-UART
Changed lines of the file:
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@@
 	(generator_version "9.0")
 	(paper "A4")
-	(text "Vcc = 3.3V\nVf = 2.2V, If = 20mA\n\n(3.3-2.2) / 0.02 = 55Ω"
+	(title_block
+		(title "GPIO Board / USB-UART")
+		(date "2025-04-03")
+		(rev "ver1.1")
+		(company "阿南高専ロボット研究部")
+	)
+	(text "Vcc = 3.3V\nVf = 2.1V, If = 12.5mA\n\n(3.3-2.1) / 0.0125 = 96Ω"
 		(exclude_from_sim no)
 		(at 184.15 124.46 0)
@@
 			)
 		)
-		(property "Name" "CL10B104KA8NNNC"
+		(property "Name" "GCJ188R91H124KA01D"
 			(at 167.64 76.2 0)
 			(effects
@@
 			)
 		)
-		(property "URL" "https://www.digikey.jp/ja/products/detail/samsung-electro-mechanics/CL10B104KA8NNNC/3886664"
+		(property "URL" "https://www.digikey.jp/ja/products/detail/murata-electronics/GCJ188R91H124KA01D/13401917"
 			(at 167.64 76.2 0)
 			(effects
@@
 			)
 		)
-		(property "Price" "12"
+		(property "Price" "36"
 			(at 167.64 76.2 0)
 			(effects
@@
 			)
 		)
-		(property "Footprint" "Diode_SMD:D_SOD-123"
+		(property "Footprint" "Diode_SMD:Nexperia_CFP3_SOD-123W"
 			(at 134.62 66.04 0)
 			(effects
@@
 			)
 		)
-		(property "Name" "RB160M-30TR"
+		(property "Name" "PMEG3010ER,115"
 			(at 134.62 66.04 0)
 			(effects
@@
 			)
 		)
-		(property "URL" "https://akizukidenshi.com/catalog/g/g101398/"
+		(property "URL" "https://www.digikey.jp/ja/products/detail/nexperia-usa-inc/PMEG3010ER-115/2119868"
 			(at 134.62 66.04 0)
 			(effects
@@
 			)
 		)
-		(property "Price" "15"
+		(property "Price" "30"
 			(at 134.62 66.04 0)
 			(effects
@@
 			)
 		)
-		(property "Value" "data"
+		(property "Value" "Data"
 			(at 181.61 113.3474 90)
 			(effects
@@
 			)
 		)
-		(property "Name" "SML-E12P8WT86"
+		(property "Name" "SML-D14MWT86A"
 			(at 177.8 110.49 0)
 			(effects
@@
 			)
 		)
-		(property "URL" "https://www.digikey.jp/ja/products/detail/rohm-semiconductor/SML-E12P8WT86/1641804"
+		(property "URL" "https://www.digikey.jp/ja/products/detail/rohm-semiconductor/SML-D14MWT86A/9448204"
 			(at 177.8 110.49 0)
 			(effects
@@
 			)
 		)
-		(property "Price" "39"
+		(property "Price" "53"
 			(at 177.8 110.49 0)
 			(effects
@@
 			)
 		)
-		(property "Name" "ESR03EZPF5101"
+		(property "Name" "ESR03EZPJ512"
 			(at 132.08 106.68 0)
 			(effects
@@
 			)
 		)
-		(property "URL" "https://www.digikey.jp/ja/products/detail/rohm-semiconductor/ESR03EZPF5101/4007250"
+		(property "URL" "https://www.digikey.jp/ja/products/detail/rohm-semiconductor/ESR03EZPJ512/1762735"
 			(at 132.08 106.68 0)
 			(effects
@@
 			)
 		)
-		(property "Price" "23"
+		(property "Price" "22"
 			(at 132.08 106.68 0)
 			(effects
@@
 			)
 		)
-		(property "Name" "ESR03EZPF5101"
+		(property "Name" "ESR03EZPJ512"
 			(at 137.16 106.68 0)
 			(effects
@@
 			)
 		)
-		(property "URL" "https://www.digikey.jp/ja/products/detail/rohm-semiconductor/ESR03EZPF5101/4007250"
+		(property "URL" "https://www.digikey.jp/ja/products/detail/rohm-semiconductor/ESR03EZPJ512/1762735"
 			(at 137.16 106.68 0)
 			(effects
@@
 			)
 		)
-		(property "Price" "23"
+		(property "Price" "22"
 			(at 137.16 106.68 0)
 			(effects
@@
 			)
 		)
-		(property "Value" "55"
+		(property "Value" "96"
 			(at 180.34 120.6499 0)
 			(effects
@@
 			)
 		)
-		(property "Name" "ESR03EZPF60R4"
+		(property "Name" "ESR03EZPJ101"
 			(at 177.8 119.38 0)
 			(effects
@@
 			)
 		)
-		(property "URL" "https://www.digikey.jp/ja/products/detail/rohm-semiconductor/ESR03EZPF60R4/20486478"
+		(property "URL" "https://www.digikey.jp/ja/products/detail/rohm-semiconductor/ESR03EZPJ101/1983452"
 			(at 177.8 119.38 0)
 			(effects
@@
 			)
 		)
-		(property "Price" "23"
+		(property "Price" "22"
 			(at 177.8 119.38 0)
 			(effects
