File: PWMBoard/PWMBoard.kicad_pcb (KiCad board)
At the start: 4 copper layers, 70 x 45 mm, 94 parts, among them J1 SWD, J10 LED1, J11 LED1, J12 BATT, J2 Debug, J3 CAN, J4 LED1, J5 LED1, J6 LED1, J7 LED1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

Commit message: PWM Board ver1.1
Connections:
- J12 pad 1: +BATT -> GNDA
- J12 pad 2: GNDA -> +BATT
Routing:
- net +BATT: track 8.94 -> 10.5 mm
- net GNDA: track 10.9 -> 11.8 mm
Other:
- board text added: "ver 1.1: 2025-06-18"
- board text removed: "ver 1.0: 2025-04-12"
