File: PWMBoard/PWMBoard.kicad_sch (KiCad schematic)
At the start: 53 parts, among them J10 LED1, J11 LED1, J12 BATT, J3 CAN, J4 LED1, J5 LED1, J6 LED1, J7 LED1, J8 LED1, J9 LED1, SW2 SW_Coded, SW3 CAN_R, U1 TLV1117-33, U7 LED_GRB, U8 TLV760

Commit message: PWM Board ver1.1
Connections:
- net +BATT: now also J12.2 (Pin_2); no longer J12.1 (Pin_1)
- net GNDA: now also J12.1 (Pin_1); no longer J12.2 (Pin_2)
- net Isolator/LED1 renamed Isolator/PWM1
- net Isolator/LED1A renamed Isolator/PWM1A
- net Isolator/LED2 renamed Isolator/PWM2
- net Isolator/LED2A renamed Isolator/PWM2A
- net Isolator/LED3 renamed Isolator/PWM3
- net Isolator/LED3A renamed Isolator/PWM3A
- net Isolator/LED4 renamed Isolator/PWM4
- net Isolator/LED4A renamed Isolator/PWM4A
- net Isolator/LED5 renamed Isolator/PWM5
- net Isolator/LED5A renamed Isolator/PWM5A
- net Isolator/LED6 renamed Isolator/PWM6
- net Isolator/LED6A renamed Isolator/PWM6A
- net Isolator/LED7 renamed Isolator/PWM7
- net Isolator/LED7A renamed Isolator/PWM7A
- net Isolator/LED8 renamed Isolator/PWM8
- net Isolator/LED8A renamed Isolator/PWM8A
Other:
- sheet CAN: file CAN.kicad_sch -> PWMBoard_CAN.kicad_sch
- sheet Isolator: file Isolator.kicad_sch -> PWMBoard_Isolator.kicad_sch
- sheet Isolator ports: added PWM1, PWM1A, PWM2, PWM2A, PWM3, PWM3A, PWM4, PWM4A, PWM5, PWM5A, PWM6, PWM6A, PWM7, PWM7A, PWM8, PWM8A; removed LED1, LED1A, LED2, LED2A, LED3, LED3A, LED4, LED4A, LED5, LED5A, LED6, LED6A, LED7, LED7A, LED8, LED8A
- sheet MCU: file MCU.kicad_sch -> PWMBoard_MCU.kicad_sch
- sheet MCU ports: added PWM1, PWM2, PWM3, PWM4, PWM5, PWM6, PWM7, PWM8; removed LED1, LED2, LED3, LED4, LED5, LED6, LED7, LED8
- sheet USB-UART: file USB-UART.kicad_sch -> PWMBoard_USB-UART.kicad_sch
- moved on the sheet: C13, C14, D16, JP2, U8
