File: PWMBoard/PWMBoard_CAN.kicad_sch (KiCad schematic)
At the start: 7 parts, among them U3 MCP2561/2FD

Commit message: PWM Board ver1.1
Changed lines of the file:
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@@
 	(title_block
 		(title "PWM Board / CAN")
-		(date "2025-04-02")
-		(rev "ver1.0")
+		(date "2025-06-18")
+		(rev "ver1.1")
 		(company "阿南高専ロボット研究部")
 	)
@@
 		)
 		(instances
-			(project "LEDBoard"
+			(project "PWMBoard"
 				(path "/24f5d1e0-9c81-4e18-bc7d-164d95be4e6f/0e3a1a86-e68f-41bc-b070-112b914674a4"
 					(reference "D3")
@@
 		)
 		(instances
-			(project "LEDBoard"
+			(project "PWMBoard"
 				(path "/24f5d1e0-9c81-4e18-bc7d-164d95be4e6f/0e3a1a86-e68f-41bc-b070-112b914674a4"
 					(reference "#PWR031")
@@
 		)
 		(instances
-			(project "LEDBoard"
+			(project "PWMBoard"
 				(path "/24f5d1e0-9c81-4e18-bc7d-164d95be4e6f/0e3a1a86-e68f-41bc-b070-112b914674a4"
 					(reference "#PWR033")
@@
 		)
 		(instances
-			(project "LEDBoard"
+			(project "PWMBoard"
 				(path "/24f5d1e0-9c81-4e18-bc7d-164d95be4e6f/0e3a1a86-e68f-41bc-b070-112b914674a4"
 					(reference "#PWR032")
@@
 		)
 		(instances
-			(project "LEDBoard"
+			(project "PWMBoard"
 				(path "/24f5d1e0-9c81-4e18-bc7d-164d95be4e6f/0e3a1a86-e68f-41bc-b070-112b914674a4"
 					(reference "R4")
@@
 		)
 		(instances
-			(project ""
+			(project "PWMBoard"
 				(path "/24f5d1e0-9c81-4e18-bc7d-164d95be4e6f/0e3a1a86-e68f-41bc-b070-112b914674a4"
 					(reference "#PWR030")
@@
 		)
 		(instances
-			(project ""
+			(project "PWMBoard"
 				(path "/24f5d1e0-9c81-4e18-bc7d-164d95be4e6f/0e3a1a86-e68f-41bc-b070-112b914674a4"
 					(reference "U3")
@@
 		)
 		(instances
-			(project ""
+			(project "PWMBoard"
 				(path "/24f5d1e0-9c81-4e18-bc7d-164d95be4e6f/0e3a1a86-e68f-41bc-b070-112b914674a4"
 					(reference "C11")
@@
 		)
 		(instances
-			(project "LEDBoard"
+			(project "PWMBoard"
 				(path "/24f5d1e0-9c81-4e18-bc7d-164d95be4e6f/0e3a1a86-e68f-41bc-b070-112b914674a4"
 					(reference "#PWR034")
@@
 		)
 		(instances
-			(project ""
+			(project "PWMBoard"
 				(path "/24f5d1e0-9c81-4e18-bc7d-164d95be4e6f/0e3a1a86-e68f-41bc-b070-112b914674a4"
 					(reference "JP1")
@@
 		)
 		(instances
-			(project ""
+			(project "PWMBoard"
 				(path "/24f5d1e0-9c81-4e18-bc7d-164d95be4e6f/0e3a1a86-e68f-41bc-b070-112b914674a4"
 					(reference "D2")
@@
 		)
 		(instances
-			(project ""
+			(project "PWMBoard"
 				(path "/24f5d1e0-9c81-4e18-bc7d-164d95be4e6f/0e3a1a86-e68f-41bc-b070-112b914674a4"
 					(reference "R3")
@@
 		(on_board yes)
 		(dnp no)
-		(fields_autoplaced yes)
 		(property "Reference" "#PWR029"
 			(at 144.78 83.82 0)
@@
 		)
 		(property "Value" "+5V"
-			(at 144.78 74.93 0)
+			(at 144.78 76.2 0)
 			(effects
 				(font
@@
 		)
 		(instances
-			(project ""
+			(project "PWMBoard"
 				(path "/24f5d1e0-9c81-4e18-bc7d-164d95be4e6f/0e3a1a86-e68f-41bc-b070-112b914674a4"
 					(reference "#PWR029")
