File: PWMBoard/PWMBoard_Isolator.kicad_sch (KiCad schematic)
At the start: 6 parts, among them U4 ISO6740, U5 ISO6740

Commit message: PWM Board ver1.1
Connections:
- net LED1 renamed PWM1
- net LED1A renamed PWM1A
- net LED2 renamed PWM2
- net LED2A renamed PWM2A
- net LED3 renamed PWM3
- net LED3A renamed PWM3A
- net LED4 renamed PWM4
- net LED4A renamed PWM4A
- net LED5 renamed PWM5
- net LED5A renamed PWM5A
- net LED6 renamed PWM6
- net LED6A renamed PWM6A
- net LED7 renamed PWM7
- net LED7A renamed PWM7A
- net LED8 renamed PWM8
- net LED8A renamed PWM8A
Changed lines of the file:
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@@
 	(title_block
 		(title "PWM Board / Isolator")
-		(date "2025-04-02")
-		(rev "ver1.0")
+		(date "2025-06-18")
+		(rev "ver1.1")
 		(company "阿南高専ロボット研究部")
 	)
@@
 		)
 	)
-	(hierarchical_label "LED6A"
+	(hierarchical_label "PWM6A"
 		(shape output)
 		(at 187.96 87.63 0)
@@
 		)
 	)
-	(hierarchical_label "LED2"
+	(hierarchical_label "PWM2"
 		(shape input)
 		(at 119.38 87.63 180)
@@
 		)
 	)
-	(hierarchical_label "LED5"
+	(hierarchical_label "PWM5"
 		(shape input)
 		(at 163.83 85.09 180)
@@
 		)
 	)
-	(hierarchical_label "LED1"
+	(hierarchical_label "PWM1"
 		(shape input)
 		(at 119.38 85.09 180)
@@
 		)
 	)
-	(hierarchical_label "LED4A"
+	(hierarchical_label "PWM4A"
 		(shape output)
 		(at 143.51 92.71 0)
@@
 		)
 	)
-	(hierarchical_label "LED1A"
+	(hierarchical_label "PWM1A"
 		(shape output)
 		(at 143.51 85.09 0)
@@
 		)
 	)
-	(hierarchical_label "LED3A"
+	(hierarchical_label "PWM3A"
 		(shape output)
 		(at 143.51 90.17 0)
@@
 		)
 	)
-	(hierarchical_label "LED6"
+	(hierarchical_label "PWM6"
 		(shape input)
 		(at 163.83 87.63 180)
@@
 		)
 	)
-	(hierarchical_label "LED5A"
+	(hierarchical_label "PWM5A"
 		(shape output)
 		(at 187.96 85.09 0)
@@
 		)
 	)
-	(hierarchical_label "LED7A"
+	(hierarchical_label "PWM7A"
 		(shape output)
 		(at 187.96 90.17 0)
@@
 		)
 	)
-	(hierarchical_label "LED7"
+	(hierarchical_label "PWM7"
 		(shape input)
 		(at 163.83 90.17 180)
@@
 		)
 	)
-	(hierarchical_label "LED3"
+	(hierarchical_label "PWM3"
 		(shape input)
 		(at 119.38 90.17 180)
@@
 		)
 	)
-	(hierarchical_label "LED8"
+	(hierarchical_label "PWM8"
 		(shape input)
 		(at 163.83 92.71 180)
@@
 		)
 	)
-	(hierarchical_label "LED8A"
+	(hierarchical_label "PWM8A"
 		(shape output)
 		(at 187.96 92.71 0)
@@
 		)
 	)
-	(hierarchical_label "LED2A"
+	(hierarchical_label "PWM2A"
 		(shape output)
 		(at 143.51 87.63 0)
@@
 		)
 	)
-	(hierarchical_label "LED4"
+	(hierarchical_label "PWM4"
 		(shape input)
 		(at 119.38 92.71 180)
@@
 		)
 		(instances
-			(project "LEDBoard"
+			(project "PWMBoard"
 				(path "/24f5d1e0-9c81-4e18-bc7d-164d95be4e6f/0775c67a-417f-4204-9522-5a26770a5c94"
 					(reference "#PWR028")
@@
 		)
 		(instances
-			(project "LEDBoard"
+			(project "PWMBoard"
 				(path "/24f5d1e0-9c81-4e18-bc7d-164d95be4e6f/0775c67a-417f-4204-9522-5a26770a5c94"
 					(reference "#PWR023")
@@
 		(on_board yes)
 		(dnp no)
-		(fields_autoplaced yes)
 		(property "Reference" "C17"
-			(at 163.8363 60.96 90)
+			(at 162.56 60.96 90)
 			(effects
 				(font
@@
 		)
 		(property "Value" "0.1u"
-			(at 163.8363 63.5 90)
+			(at 162.56 63.5 90)
 			(effects
 				(font
@@
 		)
 		(instances
-			(project "LEDBoard"
+			(project "PWMBoard"
 				(path "/24f5d1e0-9c81-4e18-bc7d-164d95be4e6f/0775c67a-417f-4204-9522-5a26770a5c94"
 					(reference "C17")
@@
 		)
 		(instances
-			(project "LEDBoard"
+			(project "PWMBoard"
 				(path "/24f5d1e0-9c81-4e18-bc7d-164d95be4e6f/0775c67a-417f-4204-9522-5a26770a5c94"
 					(reference "#PWR022")
@@
 		(on_board yes)
 		(dnp no)
-		(fields_autoplaced yes)
 		(property "Reference" "C16"
-			(at 139.7063 60.96 90)
+			(at 140.97 60.96 90)
 			(effects
 				(font
@@
 		)
 		(property "Value" "0.1u"
-			(at 139.7063 63.5 90)
+			(at 140.97 63.5 90)
 			(effects
 				(font
@@
 		)
 		(instances
-			(project "LEDBoard"
+			(project "PWMBoard"
 				(path "/24f5d1e0-9c81-4e18-bc7d-164d95be4e6f/0775c67a-417f-4204-9522-5a26770a5c94"
 					(reference "C16")
@@
 		(on_board yes)
 		(dnp no)
-		(fields_autoplaced yes)
 		(property "Reference" "#PWR026"
 			(at 179.07 71.12 0)
@@
 		)
 		(property "Value" "+5VA"
-			(at 179.07 62.23 0)
+			(at 179.07 63.5 0)
 			(effects
 				(font
@@
 		)
 		(instances
-			(project "LEDBoard"
+			(project "PWMBoard"
 				(path "/24f5d1e0-9c81-4e18-bc7d-164d95be4e6f/0775c67a-417f-4204-9522-5a26770a5c94"
 					(reference "#PWR026")
@@
 		)
 		(instances
-			(project "LEDBoard"
+			(project "PWMBoard"
 				(path "/24f5d1e0-9c81-4e18-bc7d-164d95be4e6f/0775c67a-417f-4204-9522-5a26770a5c94"
 					(reference "U5")
@@
 		(on_board yes)
 		(dnp no)
-		(fields_autoplaced yes)
 		(property "Reference" "C15"
-			(at 119.3863 60.96 90)
+			(at 118.11 60.96 90)
 			(effects
 				(font
@@
 		)
 		(property "Value" "0.1u"
-			(at 119.3863 63.5 90)
+			(at 118.11 63.5 90)
 			(effects
 				(font
@@
 		)
 		(instances
-			(project "LEDBoard"
+			(project "PWMBoard"
 				(path "/24f5d1e0-9c81-4e18-bc7d-164d95be4e6f/0775c67a-417f-4204-9522-5a26770a5c94"
 					(reference "C15")
@@
 		(on_board yes)
 		(dnp no)
-		(fields_autoplaced yes)
 		(property "Reference" "#PWR019"
 			(at 134.62 71.12 0)
@@
 		)
 		(property "Value" "+5VA"
-			(at 134.62 62.23 0)
+			(at 134.62 63.5 0)
 			(effects
 				(font
@@
 		)
 		(instances
-			(project ""
+			(project "PWMBoard"
 				(path "/24f5d1e0-9c81-4e18-bc7d-164d95be4e6f/0775c67a-417f-4204-9522-5a26770a5c94"
 					(reference "#PWR019")
@@
 		)
 		(instances
-			(project "LEDBoard"
+			(project "PWMBoard"
 				(path "/24f5d1e0-9c81-4e18-bc7d-164d95be4e6f/0775c67a-417f-4204-9522-5a26770a5c94"
 					(reference "#PWR024")
@@
 		(on_board yes)
 		(dnp no)
-		(fields_autoplaced yes)
 		(property "Reference" "C18"
-			(at 184.1563 60.96 90)
+			(at 185.42 60.96 90)
 			(effects
 				(font
@@
 		)
 		(property "Value" "0.1u"
-			(at 184.1563 63.5 90)
+			(at 185.42 63.5 90)
 			(effects
 				(font
@@
 		)
 		(instances
-			(project "LEDBoard"
+			(project "PWMBoard"
 				(path "/24f5d1e0-9c81-4e18-bc7d-164d95be4e6f/0775c67a-417f-4204-9522-5a26770a5c94"
 					(reference "C18")
@@
 		)
 		(instances
-			(project "LEDBoard"
+			(project "PWMBoard"
 				(path "/24f5d1e0-9c81-4e18-bc7d-164d95be4e6f/0775c67a-417f-4204-9522-5a26770a5c94"
 					(reference "U4")
@@
 		(on_board yes)
 		(dnp no)
-		(fields_autoplaced yes)
 		(property "Reference" "#PWR017"
 			(at 124.46 71.12 0)
@@
 		)
 		(property "Value" "+3.3V"
-			(at 124.46 62.23 0)
+			(at 124.46 63.5 0)
 			(effects
 				(font
@@
 		)
 		(instances
-			(project "LEDBoard"
+			(project "PWMBoard"
 				(path "/24f5d1e0-9c81-4e18-bc7d-164d95be4e6f/0775c67a-417f-4204-9522-5a26770a5c94"
 					(reference "#PWR017")
@@
 		)
 		(property "Value" "GNDA"
-			(at 134.62 109.474 0)
+			(at 134.62 109.22 0)
 			(effects
 				(font
@@
 		)
 		(instances
-			(project "LEDBoard"
+			(project "PWMBoard"
 				(path "/24f5d1e0-9c81-4e18-bc7d-164d95be4e6f/0775c67a-417f-4204-9522-5a26770a5c94"
 					(reference "#PWR020")
@@
 		)
 		(property "Value" "GNDA"
-			(at 179.07 109.474 0)
+			(at 179.07 109.22 0)
 			(effects
 				(font
@@
 		)
 		(instances
-			(project "LEDBoard"
+			(project "PWMBoard"
 				(path "/24f5d1e0-9c81-4e18-bc7d-164d95be4e6f/0775c67a-417f-4204-9522-5a26770a5c94"
 					(reference "#PWR027")
@@
 		)
 		(instances
-			(project "LEDBoard"
+			(project "PWMBoard"
 				(path "/24f5d1e0-9c81-4e18-bc7d-164d95be4e6f/0775c67a-417f-4204-9522-5a26770a5c94"
 					(reference "#PWR025")
@@
 		(on_board yes)
 		(dnp no)
-		(fields_autoplaced yes)
 		(property "Reference" "#PWR021"
 			(at 168.91 71.12 0)
@@
 		)
 		(property "Value" "+3.3V"
-			(at 168.91 62.23 0)
+			(at 168.91 63.5 0)
 			(effects
 				(font
@@
 		)
 		(instances
-			(project "LEDBoard"
+			(project "PWMBoard"
 				(path "/24f5d1e0-9c81-4e18-bc7d-164d95be4e6f/0775c67a-417f-4204-9522-5a26770a5c94"
 					(reference "#PWR021")
@@
 		)
 		(instances
-			(project "LEDBoard"
+			(project "PWMBoard"
 				(path "/24f5d1e0-9c81-4e18-bc7d-164d95be4e6f/0775c67a-417f-4204-9522-5a26770a5c94"
 					(reference "#PWR018")
