File: PWMBoard/PWMBoard_MCU.kicad_sch (KiCad schematic)
At the start: 15 parts, among them J1 SWD, SW1 Reset, U2 STM32F303K8Tx, Y1 Crystal_GND2

Commit message: PWM Board ver1.1
Parts:
- Y1: value Crystal_GND2 -> 32MHz
Connections:
- net LED1 renamed PWM1
- net LED2 renamed PWM2
- net LED3 renamed PWM3
- net LED4 renamed PWM4
- net LED5 renamed PWM5
- net LED6 renamed PWM6
- net LED7 renamed PWM7
- net LED8 renamed PWM8
Other:
- note added: "PWM1: PA1: TIM2_CH2 PWM2: PA2: TIM2_CH3 PWM3: PA3: TIM2_CH4 PWM4: PA5: TIM2_CH1 PWM5: PA6: TIM3_CH1 PWM6: PA7: TIM3_CH2 PWM7: PB0: TIM3_CH3 PWM8: PB1: TIM3_CH4 LED_R: TIM1_CH2 LED_G: TIM1_CH3 LED_B: TIM1_CH1 USART2_TX: PB3 USART2_RX: PA15"
- note removed: "LED1: PA1: TIM2_CH2 LED2: PA2: TIM2_CH3 LED3: PA3: TIM2_CH4 LED4: PA5: TIM2_CH1 LED5: PA6: TIM3_CH1 LED6: PA7: TIM3_CH2 LED7: PB0: TIM3_CH3 LED8: PB1: TIM3_CH4 LED_R: TIM1_CH2 LED_G: TIM1_CH3 LED_B: TIM1_CH1 USART2_TX: PB3 USART2_RX: PA15"
Changed lines of the file:
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@@
 	(title_block
 		(title "PWM Board / MCU")
-		(date "2025-04-02")
-		(rev "ver1.0")
+		(date "2025-06-18")
+		(rev "ver1.1")
 		(company "阿南高専ロボット研究部")
 	)
-	(text "LED1: PA1: TIM2_CH2\nLED2: PA2: TIM2_CH3\nLED3: PA3: TIM2_CH4\nLED4: PA5: TIM2_CH1\nLED5: PA6: TIM3_CH1\nLED6: PA7: TIM3_CH2\nLED7: PB0: TIM3_CH3\nLED8: PB1: TIM3_CH4\n\nLED_R: TIM1_CH2\nLED_G: TIM1_CH3\nLED_B: TIM1_CH1\n\nUSART2_TX: PB3\nUSART2_RX: PA15"
+	(text "PWM1: PA1: TIM2_CH2\nPWM2: PA2: TIM2_CH3\nPWM3: PA3: TIM2_CH4\nPWM4: PA5: TIM2_CH1\nPWM5: PA6: TIM3_CH1\nPWM6: PA7: TIM3_CH2\nPWM7: PB0: TIM3_CH3\nPWM8: PB1: TIM3_CH4\n\nLED_R: TIM1_CH2\nLED_G: TIM1_CH3\nLED_B: TIM1_CH1\n\nUSART2_TX: PB3\nUSART2_RX: PA15"
 		(exclude_from_sim no)
 		(at 183.642 88.9 0)
@@
 		)
 	)
-	(hierarchical_label "LED4"
+	(hierarchical_label "PWM4"
 		(shape output)
 		(at 157.48 91.44 0)
@@
 		)
 	)
-	(hierarchical_label "LED3"
+	(hierarchical_label "PWM3"
 		(shape output)
 		(at 157.48 86.36 0)
@@
 		)
 	)
-	(hierarchical_label "LED7"
+	(hierarchical_label "PWM7"
 		(shape output)
 		(at 127 96.52 180)
@@
 		)
 	)
-	(hierarchical_label "LED1"
-		(shape output)
-		(at 157.48 81.28 0)
-		(effects
-			(font
-				(size 1.27 1.27)
-			)
-			(justify left)
-		)
-	)
-	(hierarchical_label "LED5"
+	(hierarchical_label "PWM5"
 		(shape output)
 		(at 157.48 93.98 0)
@@
 		)
 	)
+	(hierarchical_label "PWM1"
+		(shape output)
+		(at 157.48 81.28 0)
+		(effects
+			(font
+				(size 1.27 1.27)
+			)
+			(justify left)
+		)
+	)
 	(hierarchical_label "CAN_RX"
 		(shape input)
@@
 		)
 	)
-	(hierarchical_label "LED8"
+	(hierarchical_label "PWM8"
 		(shape output)
 		(at 127 99.06 180)
@@
 		)
 	)
-	(hierarchical_label "LED2"
+	(hierarchical_label "PWM2"
 		(shape output)
 		(at 157.48 83.82 0)
@@
 		)
 	)
-	(hierarchical_label "LED6"
+	(hierarchical_label "PWM6"
 		(shape output)
 		(at 157.48 96.52 0)
@@
 		)
 		(instances
-			(project ""
+			(project "PWMBoard"
 				(path "/24f5d1e0-9c81-4e18-bc7d-164d95be4e6f/984e9e8d-b2d8-43fb-8904-98e9cdb015a3"
 					(reference "#PWR013")
@@
 		)
 		(instances
-			(project ""
+			(project "PWMBoard"
 				(path "/24f5d1e0-9c81-4e18-bc7d-164d95be4e6f/984e9e8d-b2d8-43fb-8904-98e9cdb015a3"
 					(reference "#PWR059")
@@
 		)
 		(instances
-			(project ""
+			(project "PWMBoard"
 				(path "/24f5d1e0-9c81-4e18-bc7d-164d95be4e6f/984e9e8d-b2d8-43fb-8904-98e9cdb015a3"
 					(reference "C3")
@@
 		)
 		(instances
-			(project "LEDBoard"
+			(project "PWMBoard"
 				(path "/24f5d1e0-9c81-4e18-bc7d-164d95be4e6f/984e9e8d-b2d8-43fb-8904-98e9cdb015a3"
 					(reference "C6")
@@
 		)
 		(instances
-			(project ""
+			(project "PWMBoard"
 				(path "/24f5d1e0-9c81-4e18-bc7d-164d95be4e6f/984e9e8d-b2d8-43fb-8904-98e9cdb015a3"
 					(reference "U2")
@@
 		(on_board yes)
 		(dnp no)
-		(fields_autoplaced yes)
 		(property "Reference" "Y1"
-			(at 102.87 91.44 0)
-			(effects
-				(font
-					(size 1.27 1.27)
-				)
-			)
-		)
-		(property "Value" "Crystal_GND2"
-			(at 102.87 93.98 0)
+			(at 102.87 92.075 0)
+			(effects
+				(font
+					(size 1.27 1.27)
+				)
+			)
+		)
+		(property "Value" "32MHz"
+			(at 102.87 94.615 0)
 			(effects
 				(font
@@
 		)
 		(instances
-			(project ""
+			(project "PWMBoard"
 				(path "/24f5d1e0-9c81-4e18-bc7d-164d95be4e6f/984e9e8d-b2d8-43fb-8904-98e9cdb015a3"
 					(reference "Y1")
@@
 		)
 		(instances
-			(project ""
+			(project "PWMBoard"
 				(path "/24f5d1e0-9c81-4e18-bc7d-164d95be4e6f/984e9e8d-b2d8-43fb-8904-98e9cdb015a3"
 					(reference "#PWR012")
@@
 		)
 		(instances
-			(project ""
+			(project "PWMBoard"
 				(path "/24f5d1e0-9c81-4e18-bc7d-164d95be4e6f/984e9e8d-b2d8-43fb-8904-98e9cdb015a3"
 					(reference "C8")
@@
 		)
 		(instances
-			(project "LEDBoard"
+			(project "PWMBoard"
 				(path "/24f5d1e0-9c81-4e18-bc7d-164d95be4e6f/984e9e8d-b2d8-43fb-8904-98e9cdb015a3"
 					(reference "C7")
@@
 		(on_board yes)
 		(dnp no)
-		(fields_autoplaced yes)
 		(property "Reference" "#PWR08"
 			(at 163.83 60.96 0)
@@
 		)
 		(property "Value" "+3.3VADC"
-			(at 160.02 54.61 0)
+			(at 160.02 55.88 0)
 			(effects
 				(font
@@
 		)
 		(instances
-			(project ""
+			(project "PWMBoard"
 				(path "/24f5d1e0-9c81-4e18-bc7d-164d95be4e6f/984e9e8d-b2d8-43fb-8904-98e9cdb015a3"
 					(reference "#PWR08")
@@
 		)
 		(instances
-			(project ""
+			(project "PWMBoard"
 				(path "/24f5d1e0-9c81-4e18-bc7d-164d95be4e6f/984e9e8d-b2d8-43fb-8904-98e9cdb015a3"
 					(reference "SW1")
@@
 		)
 		(instances
-			(project ""
+			(project "PWMBoard"
 				(path "/24f5d1e0-9c81-4e18-bc7d-164d95be4e6f/984e9e8d-b2d8-43fb-8904-98e9cdb015a3"
 					(reference "FB1")
@@
 		)
 		(instances
-			(project ""
+			(project "PWMBoard"
 				(path "/24f5d1e0-9c81-4e18-bc7d-164d95be4e6f/984e9e8d-b2d8-43fb-8904-98e9cdb015a3"
 					(reference "#PWR010")
@@
 		)
 		(instances
-			(project ""
+			(project "PWMBoard"
 				(path "/24f5d1e0-9c81-4e18-bc7d-164d95be4e6f/984e9e8d-b2d8-43fb-8904-98e9cdb015a3"
 					(reference "J1")
@@
 		)
 		(instances
-			(project ""
+			(project "PWMBoard"
 				(path "/24f5d1e0-9c81-4e18-bc7d-164d95be4e6f/984e9e8d-b2d8-43fb-8904-98e9cdb015a3"
 					(reference "#PWR011")
@@
 		)
 		(instances
-			(project ""
+			(project "PWMBoard"
 				(path "/24f5d1e0-9c81-4e18-bc7d-164d95be4e6f/984e9e8d-b2d8-43fb-8904-98e9cdb015a3"
 					(reference "C10")
@@
 		(on_board yes)
 		(dnp no)
-		(fields_autoplaced yes)
 		(property "Reference" "#PWR014"
 			(at 87.63 69.215 0)
@@
 		)
 		(property "Value" "+3.3V"
-			(at 87.63 60.325 0)
+			(at 87.63 61.595 0)
 			(effects
 				(font
@@
 		)
 		(instances
-			(project ""
+			(project "PWMBoard"
 				(path "/24f5d1e0-9c81-4e18-bc7d-164d95be4e6f/984e9e8d-b2d8-43fb-8904-98e9cdb015a3"
 					(reference "#PWR07")
@@
 		)
 		(instances
-			(project "LEDBoard"
+			(project "PWMBoard"
 				(path "/24f5d1e0-9c81-4e18-bc7d-164d95be4e6f/984e9e8d-b2d8-43fb-8904-98e9cdb015a3"
 					(reference "C4")
@@
 		)
 		(instances
-			(project "LEDBoard"
+			(project "PWMBoard"
 				(path "/24f5d1e0-9c81-4e18-bc7d-164d95be4e6f/984e9e8d-b2d8-43fb-8904-98e9cdb015a3"
 					(reference "C5")
@@
 		)
 		(instances
-			(project ""
+			(project "PWMBoard"
 				(path "/24f5d1e0-9c81-4e18-bc7d-164d95be4e6f/984e9e8d-b2d8-43fb-8904-98e9cdb015a3"
 					(reference "#PWR09")
@@
 		(on_board yes)
 		(dnp no)
-		(fields_autoplaced yes)
 		(property "Reference" "#PWR06"
 			(at 139.7 63.5 0)
@@
 		)
 		(property "Value" "+3.3V"
-			(at 139.7 54.61 0)
+			(at 139.7 55.88 0)
 			(effects
 				(font
@@
 		)
 		(instances
-			(project ""
+			(project "PWMBoard"
 				(path "/24f5d1e0-9c81-4e18-bc7d-164d95be4e6f/984e9e8d-b2d8-43fb-8904-98e9cdb015a3"
 					(reference "#PWR06")
@@
 		)
 		(instances
-			(project "LEDBoard"
+			(project "PWMBoard"
 				(path "/24f5d1e0-9c81-4e18-bc7d-164d95be4e6f/984e9e8d-b2d8-43fb-8904-98e9cdb015a3"
 					(reference "C9")
@@
 		)
 		(instances
-			(project "LEDBoard"
+			(project "PWMBoard"
 				(path "/24f5d1e0-9c81-4e18-bc7d-164d95be4e6f/984e9e8d-b2d8-43fb-8904-98e9cdb015a3"
 					(reference "#PWR015")
@@
 		)
 		(instances
-			(project "LEDBoard"
+			(project "PWMBoard"
 				(path "/24f5d1e0-9c81-4e18-bc7d-164d95be4e6f/984e9e8d-b2d8-43fb-8904-98e9cdb015a3"
 					(reference "#PWR016")
