File: PWMBoard/PWMBoard_USB-UART.kicad_sch (KiCad schematic)
At the start: 9 parts, among them J2 Debug, U6 CH340E

Commit message: PWM Board ver1.1
Parts:
- D4: value Data -> DATA
- J2: value Debug -> DEBUG
Changed lines of the file:
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@@
 	(title_block
 		(title "PWM Board / USB-UART")
-		(date "2025-04-02")
-		(rev "ver1.0")
+		(date "2025-06-18")
+		(rev "ver1.1")
 		(company "阿南高専ロボット研究部")
 	)
@@
 		)
 		(instances
-			(project ""
+			(project "PWMBoard"
 				(path "/24f5d1e0-9c81-4e18-bc7d-164d95be4e6f/df01c4eb-5b98-4717-8f2c-f5357a680fea"
 					(reference "#PWR037")
@@
 		)
 		(instances
-			(project ""
+			(project "PWMBoard"
 				(path "/24f5d1e0-9c81-4e18-bc7d-164d95be4e6f/df01c4eb-5b98-4717-8f2c-f5357a680fea"
 					(reference "R5")
@@
 		)
 		(instances
-			(project ""
+			(project "PWMBoard"
 				(path "/24f5d1e0-9c81-4e18-bc7d-164d95be4e6f/df01c4eb-5b98-4717-8f2c-f5357a680fea"
 					(reference "F1")
@@
 		)
 		(instances
-			(project "LEDBoard"
+			(project "PWMBoard"
 				(path "/24f5d1e0-9c81-4e18-bc7d-164d95be4e6f/df01c4eb-5b98-4717-8f2c-f5357a680fea"
 					(reference "#PWR039")
@@
 		)
 		(instances
-			(project ""
+			(project "PWMBoard"
 				(path "/24f5d1e0-9c81-4e18-bc7d-164d95be4e6f/df01c4eb-5b98-4717-8f2c-f5357a680fea"
 					(reference "#PWR038")
@@
 		)
 		(instances
-			(project ""
+			(project "PWMBoard"
 				(path "/24f5d1e0-9c81-4e18-bc7d-164d95be4e6f/df01c4eb-5b98-4717-8f2c-f5357a680fea"
 					(reference "U6")
@@
 			)
 		)
-		(property "Value" "Debug"
+		(property "Value" "DEBUG"
 			(at 114.3 60.96 0)
 			(effects
@@
 		)
 		(instances
-			(project ""
+			(project "PWMBoard"
 				(path "/24f5d1e0-9c81-4e18-bc7d-164d95be4e6f/df01c4eb-5b98-4717-8f2c-f5357a680fea"
 					(reference "J2")
@@
 		(on_board yes)
 		(dnp no)
-		(fields_autoplaced yes)
 		(property "Reference" "#PWR036"
 			(at 163.83 67.31 0)
@@
 		)
 		(property "Value" "+3.3V"
-			(at 163.83 58.42 0)
+			(at 163.83 59.69 0)
 			(effects
 				(font
@@
 		)
 		(instances
-			(project ""
+			(project "PWMBoard"
 				(path "/24f5d1e0-9c81-4e18-bc7d-164d95be4e6f/df01c4eb-5b98-4717-8f2c-f5357a680fea"
 					(reference "#PWR036")
@@
 		)
 		(instances
-			(project "LEDBoard"
+			(project "PWMBoard"
 				(path "/24f5d1e0-9c81-4e18-bc7d-164d95be4e6f/df01c4eb-5b98-4717-8f2c-f5357a680fea"
 					(reference "#PWR040")
@@
 		)
 		(instances
-			(project ""
+			(project "PWMBoard"
 				(path "/24f5d1e0-9c81-4e18-bc7d-164d95be4e6f/df01c4eb-5b98-4717-8f2c-f5357a680fea"
 					(reference "C12")
@@
 			)
 		)
-		(property "Value" "Data"
+		(property "Value" "DATA"
 			(at 185.42 103.1874 90)
 			(effects
@@
 		)
 		(instances
-			(project ""
+			(project "PWMBoard"
 				(path "/24f5d1e0-9c81-4e18-bc7d-164d95be4e6f/df01c4eb-5b98-4717-8f2c-f5357a680fea"
 					(reference "D4")
@@
 		)
 		(instances
-			(project ""
+			(project "PWMBoard"
 				(path "/24f5d1e0-9c81-4e18-bc7d-164d95be4e6f/df01c4eb-5b98-4717-8f2c-f5357a680fea"
 					(reference "D5")
@@
 		(on_board yes)
 		(dnp no)
-		(fields_autoplaced yes)
 		(property "Reference" "#PWR035"
 			(at 132.08 52.07 0)
@@
 		)
 		(property "Value" "+5V"
-			(at 132.08 43.18 0)
+			(at 132.08 44.45 0)
 			(effects
 				(font
@@
 		)
 		(instances
-			(project ""
+			(project "PWMBoard"
 				(path "/24f5d1e0-9c81-4e18-bc7d-164d95be4e6f/df01c4eb-5b98-4717-8f2c-f5357a680fea"
 					(reference "#PWR035")
@@
 		)
 		(instances
-			(project "LEDBoard"
+			(project "PWMBoard"
 				(path "/24f5d1e0-9c81-4e18-bc7d-164d95be4e6f/df01c4eb-5b98-4717-8f2c-f5357a680fea"
 					(reference "R7")
@@
 		)
 		(instances
-			(project "LEDBoard"
+			(project "PWMBoard"
 				(path "/24f5d1e0-9c81-4e18-bc7d-164d95be4e6f/df01c4eb-5b98-4717-8f2c-f5357a680fea"
 					(reference "#PWR042")
@@
 		)
 		(instances
-			(project "LEDBoard"
+			(project "PWMBoard"
 				(path "/24f5d1e0-9c81-4e18-bc7d-164d95be4e6f/df01c4eb-5b98-4717-8f2c-f5357a680fea"
 					(reference "R6")
@@
 		)
 		(instances
-			(project "LEDBoard"
+			(project "PWMBoard"
 				(path "/24f5d1e0-9c81-4e18-bc7d-164d95be4e6f/df01c4eb-5b98-4717-8f2c-f5357a680fea"
 					(reference "#PWR041")
