File: SolenoidDriver/SolenoidDriver.kicad_pcb (KiCad board)
At the start: 4 copper layers, 70 x 45 mm, 121 parts, among them J1 SWD, J10 SOL4A, J11 SOL4B, J12 BATT, J2 Debug, J3 CAN, J4 SOL1A, J5 SOL1B, J6 SOL2A, J7 SOL2B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

Commit message: Solenoid Driver ver1.1
Parts:
- added R37: 20, Resistor_SMD:R_0603_1608Metric, B.Cu at (209.6, 121.8)
- added R38: 20, Resistor_SMD:R_0603_1608Metric, B.Cu at (216.1, 121.8)
- added R39: 20, Resistor_SMD:R_0603_1608Metric, B.Cu at (222.6, 121.8)
- added R40: 20, Resistor_SMD:R_0603_1608Metric, B.Cu at (229.1, 121.8)
- added R41: 20, Resistor_SMD:R_0603_1608Metric, B.Cu at (238.7, 123.8)
- added R42: 20, Resistor_SMD:R_0603_1608Metric, B.Cu at (238.7, 130.3)
- added R43: 20, Resistor_SMD:R_0603_1608Metric, B.Cu at (238.7, 136.8)
- added R44: 20, Resistor_SMD:R_0603_1608Metric, B.Cu at (238.7, 143.3)
- moved C3 70.7 mm to (214.1, 141.9)
- moved C8 70.7 mm to (218.8, 135.1)
- moved D1 70.7 mm to (203.9, 152.9)
- moved D2 70.7 mm to (194.5, 152.9)
- moved R52 70.7 mm to (206.4, 150.9)
- moved R60 70.7 mm to (236.2, 146.6)
- moved SW3 70.7 mm to (222.6, 141.4)
- moved C1 70.7 mm to (204.1, 148.2)
- moved C10 70.7 mm to (218.4, 138.1)
- moved C11 70.7 mm to (183.1, 140.1)
- moved C12 70.7 mm to (198.6, 136.1)
- moved C2 70.7 mm to (204.1, 144.8)
- moved C4 70.7 mm to (201.1, 132.1)
- moved C6 70.7 mm to (213.6, 135.1)
- moved C7 70.7 mm to (215.3, 135.1)
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Connections:
- J12 pad 1: +BATT -> GNDA
- J12 pad 2: GNDA -> +BATT
- Q1 pad 5: /MOSFET/SOL1B- -> Net-(Q1B-D-Pad5)
- Q1 pad 6: /MOSFET/SOL1B- -> Net-(Q1B-D-Pad5)
- Q1 pad 7: /MOSFET/SOL1A- -> Net-(Q1A-D-Pad7)
- Q1 pad 8: /MOSFET/SOL1A- -> Net-(Q1A-D-Pad7)
- Q2 pad 5: /MOSFET/SOL2B- -> Net-(Q2B-D-Pad5)
- Q2 pad 6: /MOSFET/SOL2B- -> Net-(Q2B-D-Pad5)
- Q2 pad 7: /MOSFET/SOL2A- -> Net-(Q2A-D-Pad7)
- Q2 pad 8: /MOSFET/SOL2A- -> Net-(Q2A-D-Pad7)
- Q3 pad 5: /MOSFET/SOL3B- -> Net-(Q3B-D-Pad5)
- Q3 pad 6: /MOSFET/SOL3B- -> Net-(Q3B-D-Pad5)
- Q3 pad 7: /MOSFET/SOL3A- -> Net-(Q3A-D-Pad7)
- Q3 pad 8: /MOSFET/SOL3A- -> Net-(Q3A-D-Pad7)
- Q4 pad 5: /MOSFET/SOL4B- -> Net-(Q4B-D-Pad5)
- Q4 pad 6: /MOSFET/SOL4B- -> Net-(Q4B-D-Pad5)
- Q4 pad 7: /MOSFET/SOL4A- -> Net-(Q4A-D-Pad7)
- Q4 pad 8: /MOSFET/SOL4A- -> Net-(Q4A-D-Pad7)
Routing:
- net Net-(Q3A-D-Pad7): track 0.00 -> 9.46 mm, vias 0 -> 3
- net /MOSFET/SOL3A-: track 16.6 -> 7.26 mm, vias 2 -> 0
- net /MOSFET/SOL2B-: track 15.7 -> 7.26 mm, vias 2 -> 0
- net /MOSFET/SOL4B-: track 15.0 -> 7.26 mm, vias 2 -> 0
- net Net-(Q2B-D-Pad5): track 0.00 -> 7.73 mm, vias 0 -> 3
- net /MOSFET/SOL1A-: track 14.9 -> 7.21 mm, vias 2 -> 0
- net Net-(Q1A-D-Pad7): track 0.00 -> 7.19 mm, vias 0 -> 3
- net /MOSFET/SOL2A-: track 14.1 -> 7.26 mm, vias 2 -> 0
- net /MOSFET/SOL3B-: track 14.0 -> 7.26 mm, vias 2 -> 0
- net /MOSFET/SOL4A-: track 14.0 -> 7.26 mm, vias 2 -> 0
- net Net-(Q3B-D-Pad5): track 0.00 -> 6.71 mm, vias 0 -> 3
- net Net-(Q4B-D-Pad5): track 0.00 -> 6.70 mm, vias 0 -> 3
- net /MOSFET/SOL1B-: track 13.2 -> 7.26 mm, vias 2 -> 0
- net Net-(Q4A-D-Pad7): track 0.00 -> 5.87 mm, vias 0 -> 3
- net Net-(Q2A-D-Pad7): track 0.00 -> 5.77 mm, vias 0 -> 3
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Other:
- outline, holes or cut-outs redrawn
- board text added: "5V"
- board text added: "CAN-H"
- board text added: "CAN-L"
- board text added: "GND"
- board text added: "ver 1.1: 2025-07-01"
- board text removed: "ver 1.0: 2025-04-12"
