File: SolenoidDriver/SolenoidDriver.kicad_sch (KiCad schematic)
At the start: 52 parts, among them J10 SOL4A, J11 SOL4B, J12 BATT, J3 CAN, J4 SOL1A, J5 SOL1B, J6 SOL2A, J7 SOL2B, J8 SOL3A, J9 SOL3B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

Commit message: Solenoid Driver ver1.1
Connections:
- net +BATT: now also J12.2 (Pin_2); no longer J12.1 (Pin_1)
- net GNDA: now also J12.1 (Pin_1); no longer J12.2 (Pin_2)
Other:
- sheet CAN: file CAN.kicad_sch -> SolenoidDriver_CAN.kicad_sch
- sheet Isolator: file Isolator.kicad_sch -> SolenoidDriver_Isolator.kicad_sch
- sheet MCU: file MCU.kicad_sch -> SolenoidDriver_MCU.kicad_sch
- sheet MOSFET: file MOSFET.kicad_sch -> SolenoidDriver_MOSFET.kicad_sch
- sheet USB-UART: file USB-UART.kicad_sch -> SolenoidDriver_USB-UART.kicad_sch
- moved on the sheet: J12
Changed lines of the file:
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@@
 	(title_block
 		(title "Solenoid Driver")
-		(date "2025-04-08")
-		(rev "ver1.0")
+		(date "2025-07-01")
+		(rev "ver1.1")
 		(company "阿南高専ロボット研究部")
 	)
@@
 	(symbol
 		(lib_id "Connector_Generic:Conn_01x02")
-		(at 237.49 120.65 0)
-		(mirror y)
+		(at 237.49 123.19 180)
 		(unit 1)
 		(exclude_from_sim no)
@@
 		(dnp no)
 		(property "Reference" "J12"
-			(at 234.315 120.6499 0)
+			(at 234.315 123.1901 0)
 			(effects
 				(font
@@
 		)
 		(property "Value" "BATT"
-			(at 234.315 123.1899 0)
+			(at 234.315 120.6501 0)
 			(effects
 				(font
@@
 		)
 		(property "Footprint" "Connector_AMASS:AMASS_XT30PW-M_1x02_P2.50mm_Horizontal"
-			(at 237.49 120.65 0)
+			(at 237.49 123.19 0)
 			(effects
 				(font
@@
 		)
 		(property "Datasheet" "~"
-			(at 237.49 120.65 0)
+			(at 237.49 123.19 0)
 			(effects
 				(font
@@
 		)
 		(property "Description" "Generic connector, single row, 01x02, script generated (kicad-library-utils/schlib/autogen/connector/)"
-			(at 237.49 120.65 0)
+			(at 237.49 123.19 0)
 			(effects
 				(font
@@
 		)
 		(property "Name" "XT30PW-M"
-			(at 237.49 120.65 0)
+			(at 237.49 123.19 0)
 			(effects
 				(font
@@
 		)
 		(property "URL" "https://akizukidenshi.com/catalog/g/g117949/"
-			(at 237.49 120.65 0)
+			(at 237.49 123.19 0)
 			(effects
 				(font
@@
 		)
 		(property "Price" "70"
-			(at 237.49 120.65 0)
+			(at 237.49 123.19 0)
 			(effects
 				(font
@@
 		)
 		(instances
-			(project ""
+			(project "SolenoidDriver"
 				(path "/3bf18fb8-b9ed-4738-a3ef-04c20715e6dc"
 					(reference "J12")
@@
 			)
 		)
-		(property "Sheetfile" "Isolator.kicad_sch"
+		(property "Sheetfile" "SolenoidDriver_Isolator.kicad_sch"
 			(at 208.28 99.6446 0)
 			(effects
@@
 			)
 		)
-		(property "Sheetfile" "CAN.kicad_sch"
+		(property "Sheetfile" "SolenoidDriver_CAN.kicad_sch"
 			(at 74.93 57.7346 0)
 			(effects
@@
 			)
 		)
-		(property "Sheetfile" "USB-UART.kicad_sch"
+		(property "Sheetfile" "SolenoidDriver_USB-UART.kicad_sch"
 			(at 74.93 90.7546 0)
 			(effects
@@
 			)
 		)
-		(property "Sheetfile" "MOSFET.kicad_sch"
+		(property "Sheetfile" "SolenoidDriver_MOSFET.kicad_sch"
 			(at 241.3 99.6446 0)
 			(effects
@@
 			)
 		)
-		(property "Sheetfile" "MCU.kicad_sch"
+		(property "Sheetfile" "SolenoidDriver_MCU.kicad_sch"
 			(at 107.95 145.3646 0)
 			(effects
