File: RoboMasterBoard/RoboMasterBoard.kicad_pcb (KiCad board)
At the start: 2 copper layers, 70 x 45 mm, 89 parts, among them J1 SWD, J10 RM7, J11 RM8, J2 CAN1, J3 Debug, J4 RM1, J5 RM2, J6 RM3, J7 RM4, J8 RM5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

Commit message: RoboMaster Board ver1.1
Routing:
- net GNDD: track 13.7 -> 16.3 mm, vias 35 -> 38
Other:
- board text added: "ver 1.1: 2025-07-01"
- board text removed: "ver 1.0: 2025-04-12"
