File: RoboMasterBoard/RoboMasterBoard.kicad_sch (KiCad schematic)
At the start: 47 parts, among them J10 RM7, J11 RM8, J2 CAN1, J4 RM1, J5 RM2, J6 RM3, J7 RM4, J8 RM5, J9 RM6, SW2 CAN_R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

Commit message: RoboMaster Board ver1.1
Other:
- sheet CAN1: file CAN1.kicad_sch -> RoboMasterBoard_CAN1.kicad_sch
- sheet CAN2: file CAN2.kicad_sch -> RoboMasterBoard_CAN2.kicad_sch
- sheet MCU: file MCU.kicad_sch -> RoboMasterBoard_MCU.kicad_sch
- sheet USB: file USB.kicad_sch -> RoboMasterBoard_USB.kicad_sch
Changed lines of the file:
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@@
 	(title_block
 		(title "RoboMaster Board")
-		(date "2025-04-03")
-		(rev "ver1.0")
+		(date "2025-07-01")
+		(rev "ver1.1")
 		(company "阿南高専ロボット研究部")
 	)
@@
 			)
 		)
-		(property "Sheetfile" "CAN2.kicad_sch"
+		(property "Sheetfile" "RoboMasterBoard_CAN2.kicad_sch"
 			(at 142.24 57.7346 0)
 			(effects
@@
 			)
 		)
-		(property "Sheetfile" "CAN1.kicad_sch"
+		(property "Sheetfile" "RoboMasterBoard_CAN1.kicad_sch"
 			(at 80.01 57.7346 0)
 			(effects
@@
 			)
 		)
-		(property "Sheetfile" "USB.kicad_sch"
+		(property "Sheetfile" "RoboMasterBoard_USB.kicad_sch"
 			(at 80.01 86.9446 0)
 			(effects
@@
 			)
 		)
-		(property "Sheetfile" "MCU.kicad_sch"
+		(property "Sheetfile" "RoboMasterBoard_MCU.kicad_sch"
 			(at 106.68 145.3646 0)
 			(effects
