File: RoboMasterBoard/RoboMasterBoard_CAN1.kicad_sch (KiCad schematic)
At the start: 7 parts, among them U4 MCP2561/2FD

Commit message: RoboMaster Board ver1.1
Parts:
- removed C15: 0.1u, Capacitor_SMD:C_0603_1608Metric, symbol Device:C_Small
- removed D12: CAN_TX, LED_SMD:LED_0603_1608Metric, symbol Device:LED
- removed D13: CAN_RX, LED_SMD:LED_0603_1608Metric, symbol Device:LED
- removed JP2: SolderJumper_2_Open, Jumper:SolderJumper-2_P1.3mm_Open_Pad1.0x1.5mm, symbol Jumper:SolderJumper_2_Open
- removed R13, R14: 96, Resistor_SMD:R_0603_1608Metric, symbol Device:R
- removed U4: MCP2561/2FD, Package_SO:SOIC-8_3.9x4.9mm_P1.27mm, symbol Anan-Robo_Symbol_Library:MCP2561/2FD
- added C14: 0.1u, Capacitor_SMD:C_0603_1608Metric, symbol Device:C_Small
- added D10: CAN_TX, LED_SMD:LED_0603_1608Metric, symbol Device:LED
- added D11: CAN_RX, LED_SMD:LED_0603_1608Metric, symbol Device:LED
- added JP1: SolderJumper_2_Open, Jumper:SolderJumper-2_P1.3mm_Open_Pad1.0x1.5mm, symbol Jumper:SolderJumper_2_Open
- added R11, R12: 96, Resistor_SMD:R_0603_1608Metric, symbol Device:R
- added U3: MCP2561/2FD, Package_SO:SOIC-8_3.9x4.9mm_P1.27mm, symbol Anan-Robo_Symbol_Library:MCP2561/2FD
Connections:
- net +5V: now also C14.1, JP1.2 (B), U3.3 (VDD)
- net CAN_H: now also U3.7 (CANH)
- net CAN_L: now also U3.6 (CANL)
- net CAN_RX: now also D11.2 (A), U3.4 (RXD)
- net CAN_TX: now also D10.2 (A), U3.1 (TXD)
- net GNDD: now also C14.2, R11.2, R12.2, U3.2 (VSS), U3.8 (STBY)
- new net: D11.1 (K), R12.1
- new net: D10.1 (K), R11.1
- new net: JP1.1 (A), U3.5 (VIO)
Other:
- title: RoboMaster Board / CAN2 -> RoboMaster Board / CAN1
