File: RoboMasterBoard/RoboMasterBoard_CAN2.kicad_sch (KiCad schematic)
At the start: 7 parts, among them U3 MCP2561/2FD

Commit message: RoboMaster Board ver1.1
Parts:
- removed C14: 0.1u, Capacitor_SMD:C_0603_1608Metric, symbol Device:C_Small
- removed D10: CAN_TX, LED_SMD:LED_0603_1608Metric, symbol Device:LED
- removed D11: CAN_RX, LED_SMD:LED_0603_1608Metric, symbol Device:LED
- removed JP1: SolderJumper_2_Open, Jumper:SolderJumper-2_P1.3mm_Open_Pad1.0x1.5mm, symbol Jumper:SolderJumper_2_Open
- removed R11, R12: 96, Resistor_SMD:R_0603_1608Metric, symbol Device:R
- removed U3: MCP2561/2FD, Package_SO:SOIC-8_3.9x4.9mm_P1.27mm, symbol Anan-Robo_Symbol_Library:MCP2561/2FD
- added C15: 0.1u, Capacitor_SMD:C_0603_1608Metric, symbol Device:C_Small
- added D12: CAN_TX, LED_SMD:LED_0603_1608Metric, symbol Device:LED
- added D13: CAN_RX, LED_SMD:LED_0603_1608Metric, symbol Device:LED
- added JP2: SolderJumper_2_Open, Jumper:SolderJumper-2_P1.3mm_Open_Pad1.0x1.5mm, symbol Jumper:SolderJumper_2_Open
- added R13, R14: 96, Resistor_SMD:R_0603_1608Metric, symbol Device:R
- added U4: MCP2561/2FD, Package_SO:SOIC-8_3.9x4.9mm_P1.27mm, symbol Anan-Robo_Symbol_Library:MCP2561/2FD
Connections:
- net +5V: now also C15.1, JP2.2 (B), U4.3 (VDD)
- net CAN_H: now also U4.7 (CANH)
- net CAN_L: now also U4.6 (CANL)
- net CAN_RX: now also D13.2 (A), U4.4 (RXD)
- net CAN_TX: now also D12.2 (A), U4.1 (TXD)
- net GNDD: now also C15.2, R13.2, R14.2, U4.2 (VSS), U4.8 (STBY)
- new net: D13.1 (K), R14.1
- new net: D12.1 (K), R13.1
- new net: JP2.1 (A), U4.5 (VIO)
Other:
- title: RoboMaster Board / CAN1 -> RoboMaster Board / CAN2
