File: RoboMasterBoard/RoboMasterBoard_MCU.kicad_sch (KiCad schematic)
At the start: 18 parts, among them J1 SWD, SW1 RESET, U2 STM32F446RETx, Y1 Crystal_GND2

Commit message: RoboMaster Board ver1.1
Parts:
- Y1: Name XRCGB32M000F1SADR0 -> XRCGB26M000F1SADR0; Price 52 -> 50; URL https://www.digikey.jp/ja/products/detail/murata-electronics/XRCGB32M000F1SADR0/21662918?s=N4IgTCBcDaIBoCUDCBxAQgZjAWQAz4DEBGAZQEEARBXEAXQF8g -> https://www.digikey.jp/ja/products/detail/murata-electronics/XRCGB26M000F1SADR0/21662900?s=N4IgTCBcDaIBoCUDCBxAQmAbAWQAz4DEBGAZQEEARBXEAXQF8g
Changed lines of the file:
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@@
 	(title_block
 		(title "RoboMaster Board / MCU")
-		(date "2025-04-03")
-		(rev "ver1.0")
+		(date "2025-07-01")
+		(rev "ver1.1")
 		(company "阿南高専ロボット研究部")
 	)
@@
 		)
 		(instances
-			(project ""
+			(project "RoboMasterBoard"
 				(path "/536c055c-dac1-48c2-8773-453985c28c73/d37e277e-f189-4ce6-8495-a58925f22be0"
 					(reference "R10")
@@
 		)
 		(instances
-			(project ""
+			(project "RoboMasterBoard"
 				(path "/536c055c-dac1-48c2-8773-453985c28c73/d37e277e-f189-4ce6-8495-a58925f22be0"
 					(reference "#PWR06")
@@
 		)
 		(instances
-			(project ""
+			(project "RoboMasterBoard"
 				(path "/536c055c-dac1-48c2-8773-453985c28c73/d37e277e-f189-4ce6-8495-a58925f22be0"
 					(reference "#PWR011")
@@
 		)
 		(instances
-			(project ""
+			(project "RoboMasterBoard"
 				(path "/536c055c-dac1-48c2-8773-453985c28c73/d37e277e-f189-4ce6-8495-a58925f22be0"
 					(reference "J1")
@@
 		)
 		(instances
-			(project ""
+			(project "RoboMasterBoard"
 				(path "/536c055c-dac1-48c2-8773-453985c28c73/d37e277e-f189-4ce6-8495-a58925f22be0"
 					(reference "#PWR012")
@@
 		)
 		(instances
-			(project ""
+			(project "RoboMasterBoard"
 				(path "/536c055c-dac1-48c2-8773-453985c28c73/d37e277e-f189-4ce6-8495-a58925f22be0"
 					(reference "#PWR09")
@@
 		)
 		(instances
-			(project ""
+			(project "RoboMasterBoard"
 				(path "/536c055c-dac1-48c2-8773-453985c28c73/d37e277e-f189-4ce6-8495-a58925f22be0"
 					(reference "#PWR08")
@@
 		)
 		(instances
-			(project ""
+			(project "RoboMasterBoard"
 				(path "/536c055c-dac1-48c2-8773-453985c28c73/d37e277e-f189-4ce6-8495-a58925f22be0"
 					(reference "FB1")
@@
 		)
 		(instances
-			(project ""
+			(project "RoboMasterBoard"
 				(path "/536c055c-dac1-48c2-8773-453985c28c73/d37e277e-f189-4ce6-8495-a58925f22be0"
 					(reference "#PWR07")
@@
 		)
 		(instances
-			(project ""
+			(project "RoboMasterBoard"
 				(path "/536c055c-dac1-48c2-8773-453985c28c73/d37e277e-f189-4ce6-8495-a58925f22be0"
 					(reference "#PWR010")
@@
 		)
 		(instances
-			(project ""
+			(project "RoboMasterBoard"
 				(path "/536c055c-dac1-48c2-8773-453985c28c73/d37e277e-f189-4ce6-8495-a58925f22be0"
 					(reference "#PWR013")
@@
 		)
 		(instances
-			(project ""
+			(project "RoboMasterBoard"
 				(path "/536c055c-dac1-48c2-8773-453985c28c73/d37e277e-f189-4ce6-8495-a58925f22be0"
 					(reference "U2")
@@
 		)
 		(instances
-			(project ""
+			(project "RoboMasterBoard"
 				(path "/536c055c-dac1-48c2-8773-453985c28c73/d37e277e-f189-4ce6-8495-a58925f22be0"
 					(reference "C3")
@@
 		)
 		(instances
-			(project ""
+			(project "RoboMasterBoard"
 				(path "/536c055c-dac1-48c2-8773-453985c28c73/d37e277e-f189-4ce6-8495-a58925f22be0"
 					(reference "R23")
@@
 		)
 		(instances
-			(project ""
+			(project "RoboMasterBoard"
 				(path "/536c055c-dac1-48c2-8773-453985c28c73/d37e277e-f189-4ce6-8495-a58925f22be0"
 					(reference "C13")
@@
 			)
 		)
-		(property "Name" "XRCGB32M000F1SADR0"
+		(property "Name" "XRCGB26M000F1SADR0"
 			(at 90.17 77.47 0)
 			(effects
@@
 			)
 		)
-		(property "URL" "https://www.digikey.jp/ja/products/detail/murata-electronics/XRCGB32M000F1SADR0/21662918?s=N4IgTCBcDaIBoCUDCBxAQgZjAWQAz4DEBGAZQEEARBXEAXQF8g"
+		(property "URL" "https://www.digikey.jp/ja/products/detail/murata-electronics/XRCGB26M000F1SADR0/21662900?s=N4IgTCBcDaIBoCUDCBxAQmAbAWQAz4DEBGAZQEEARBXEAXQF8g"
 			(at 90.17 77.47 0)
 			(effects
@@
 			)
 		)
-		(property "Price" "52"
+		(property "Price" "50"
 			(at 90.17 77.47 0)
 			(effects

Commit message: コンデンサの容量を修正
Parts:
- C10, C11: value 15p -> 12p; Name GCM1885C2A150JA16D -> GCM1885C2A120JA16D; Price 16 -> 15; URL https://www.digikey.jp/ja/products/detail/murata-electronics/GCM1885C2A150JA16D/1765189 -> https://www.digikey.jp/ja/products/detail/murata-electronics/GCM1885C2A120JA16D/2591683
- Y1: value Crystal_GND2 -> 26MHz
Changed lines of the file:
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@@
 			)
 		)
-		(property "Value" "15p"
+		(property "Value" "12p"
 			(at 97.79 82.5562 0)
 			(effects
@@
 			)
 		)
-		(property "Name" "GCM1885C2A150JA16D"
+		(property "Name" "GCM1885C2A120JA16D"
 			(at 95.25 81.28 0)
 			(effects
@@
 			)
 		)
-		(property "URL" "https://www.digikey.jp/ja/products/detail/murata-electronics/GCM1885C2A150JA16D/1765189"
+		(property "URL" "https://www.digikey.jp/ja/products/detail/murata-electronics/GCM1885C2A120JA16D/2591683"
 			(at 95.25 81.28 0)
 			(effects
@@
 			)
 		)
-		(property "Price" "16"
+		(property "Price" "15"
 			(at 95.25 81.28 0)
 			(effects
@@
 			)
 		)
-		(property "Value" "Crystal_GND2"
+		(property "Value" "26MHz"
 			(at 90.17 72.39 0)
 			(effects
@@
 			)
 		)
-		(property "Value" "15p"
+		(property "Value" "12p"
 			(at 82.804 82.55 0)
 			(effects
@@
 			)
 		)
-		(property "Name" "GCM1885C2A150JA16D"
+		(property "Name" "GCM1885C2A120JA16D"
 			(at 85.09 81.28 0)
 			(effects
@@
 			)
 		)
-		(property "URL" "https://www.digikey.jp/ja/products/detail/murata-electronics/GCM1885C2A150JA16D/1765189"
+		(property "URL" "https://www.digikey.jp/ja/products/detail/murata-electronics/GCM1885C2A120JA16D/2591683"
 			(at 85.09 81.28 0)
 			(effects
@@
 			)
 		)
-		(property "Price" "16"
+		(property "Price" "15"
 			(at 85.09 81.28 0)
 			(effects
