File: CANBusHub/CANBusHub.kicad_pcb (KiCad board)
At the start: 2 copper layers, 100 x 57 mm, 28 parts, among them J1 CAN1_IN, J11 PWR_IN, J2 CAN2_IN, J3 CAN_OUT1, J4 CAN_OUT2, J5 CAN_OUT3, J6 CAN_OUT4, J7 CAN1_OUT, J8 CAN2_OUT, SW1 CAN1/2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

Commit message: CAN Bus Hub ver1.1
Parts:
- J7, J8: moved to B.Cu
- moved J8 32.0 mm to (202.2, 96.5), turned to -90 degrees
- moved H4 21.3 mm to (203.8, 87.5)
- moved SW1 18.1 mm to (130.1, 120.5)
- moved SW5 18.1 mm to (130.1, 120.5)
- moved SW2 18.1 mm to (152.6, 120.5)
- moved SW3 18.1 mm to (175.1, 120.5)
- moved SW4 18.1 mm to (197.6, 120.5)
- moved SW6 18.1 mm to (152.6, 120.5)
- moved SW7 18.1 mm to (175.1, 120.5)
- moved SW8 18.1 mm to (197.6, 120.5)
- moved H7 15.3 mm to (110.6, 122.5), turned to 90 degrees
- moved J7 11.0 mm to (202.2, 107.0), turned to -90 degrees
- moved J1 10.5 mm to (130.7, 92.2)
- moved J2 10.5 mm to (120.2, 92.2)
- moved J3 4.40 mm to (117.6, 118.0)
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Routing:
- net +5VD: track 177.1 -> 210.3 mm
- net /CAN2_L: track 140.1 -> 163.5 mm
- net /CAN2_H: track 147.0 -> 165.9 mm, vias 5 -> 4
- net /CAN1_L: track 126.5 -> 139.7 mm
- net /CAN1_H: track 131.4 -> 137.1 mm
- net Net-(J3-Pin_3): track 13.8 -> 10.7 mm
- net Net-(J5-Pin_4): track 10.6 -> 13.7 mm
- net Net-(J6-Pin_4): track 10.6 -> 13.6 mm
- net Net-(J4-Pin_4): track 10.6 -> 13.6 mm
- net Net-(J6-Pin_3): track 13.5 -> 10.7 mm
- net Net-(J5-Pin_3): track 13.5 -> 10.7 mm
- net Net-(J4-Pin_3): track 13.5 -> 10.7 mm
- net Net-(J3-Pin_4): track 10.8 -> 13.6 mm
- net GNDD: vias 14 -> 17
Other:
- outline, holes or cut-outs redrawn
- board text added: "1"
- board text added: "2"
- board text added: "3"
- board text added: "4"
- board text added: "ver 1.1: 2025-07-13"
- board text added: "▲"
- board text removed: "ver 1.0: 2025-05-30"
