File: MotorDriver/MotorDriver.kicad_sch (KiCad schematic)
At the start: 47 parts, among them J1 VIN, J2 INPUT, M1 Motor_DC, Q1 Q_NMOS_GDS, Q2 Q_NMOS_GDS, Q3 Q_NMOS_GDS, Q4 Q_NMOS_GDS, U1 IR2302, U2 IR2302, U3 74HC00, U4 TLP2348, U5 TLP2348, U6 NJM7812SDL1

Commit message: Motor Driver ver2.0
Parts:
- removed C1, C2: 2.5u, Capacitor_SMD:C_0603_1608Metric, symbol Device:C
- removed C12: 1u, Capacitor_SMD:C_0603_1608Metric, symbol Device:C
- removed C3, C5, C8, C9: 0.1u, Capacitor_SMD:C_0603_1608Metric, symbol Device:C_Small
- removed D1, D2: D_Schottky, Diode_SMD:D_SOD-123, symbol Device:D_Schottky
- removed J2: INPUT, Anan-Robo_Footprint_Library:PAコネクタ(4ピンサイド型), symbol Connector_Generic:Conn_01x04
- removed M1: Motor_DC, Anan-Robo_Footprint_Library:XT60PW-F_Horizontal, symbol Motor:Motor_DC
- removed Q1, Q2, Q3, Q4: Q_NMOS_GDS, Package_TO_SOT_SMD:TO-252-2, symbol Device:Q_NMOS_GDS
- removed R11, R12: 175, Resistor_SMD:R_0603_1608Metric, symbol Device:R
- removed R13, R14, R15: 80, Resistor_SMD:R_0603_1608Metric, symbol Device:R
- removed U1, U2: IR2302, Package_SO:SOIC-8_3.9x4.9mm_P1.27mm, symbol Driver_FET:IR2302
- removed U3: 74HC00, Anan-Robo_Footprint_Library:SOP14, symbol 74xx:74HC00
- removed U4, U5: TLP2348, Package_SO:SO-5-6_4.55x3.7mm_P1.27mm, symbol Anan-Robo_Symbol_Library:TLP2348
- added C2: 4.7u, Capacitor_SMD:C_0603_1608Metric, symbol Device:C_Small
- added D1: D, Diode_SMD:Nexperia_CFP3_SOD-123W, symbol Device:D
- added D2: CAN_R, LED_SMD:LED_0603_1608Metric, symbol Device:LED
- added F1: Polyfuse, Anan-Robo_Footprint_Library:MF-FSMF, symbol Device:Polyfuse
- added H1, H2, H3, H4: MountingHole_Pad, MountingHole:MountingHole_3.2mm_M3_Pad, symbol Mechanical:MountingHole_Pad
- added H5: MountingHole, Anan-Robo_Footprint_Library:Title, symbol Mechanical:MountingHole
- added H6: MountingHole, Anan-Robo_Footprint_Library:Aho_old_S, symbol Mechanical:MountingHole
- added H7: MountingHole, Anan-Robo_Footprint_Library:Aho_new_S, symbol Mechanical:MountingHole
- added H8: MountingHole, Anan-Robo_Footprint_Library:Info_M_3, symbol Mechanical:MountingHole
- added J1: CAN, Connector_IDC:IDC-Header_2x03_P2.54mm_Horizontal, symbol Connector_Generic:Conn_02x03_Odd_Even
- added J2: ENC, Anan-Robo_Footprint_Library:SM05B-PASS-TBx, symbol Connector_Generic:Conn_01x05
- added J3: SW1, Anan-Robo_Footprint_Library:SM02B-PASS-TBx, symbol Connector_Generic:Conn_01x02
- added J4: SW2, Anan-Robo_Footprint_Library:SM02B-PASS-TBx, symbol Connector_Generic:Conn_01x02
- added J6: Motor, Anan-Robo_Footprint_Library:XT60PW-F_Horizontal, symbol Connector_Generic:Conn_01x02
- added JP1: Up/Down, Jumper:SolderJumper-3_P1.3mm_Open_Pad1.0x1.5mm, symbol Jumper:SolderJumper_3_Open
- added SW1: CAN_R, Anan-Robo_Footprint_Library:SLW, symbol Switch:SW_DPDT_x2
- added SW2: SW_Coded, Anan-Robo_Footprint_Library:RDS-1055-SMT, symbol Switch:SW_Coded
- added U1: LED_GRB, LED_SMD:LED_ROHM_SMLVN6, symbol Anan-Robo_Symbol_Library:LED_GRB
- added U3: TLV1117-33, Package_TO_SOT_SMD:SOT-223-3_TabPin2, symbol Regulator_Linear:TLV1117-33
- C1: renamed from C6; Name GRM188R71C474KA88D -> CL10A225KB8NNNC; Price 16 -> 37; URL https://www.digikey.jp/ja/products/detail/murata-electronic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 -> https://www.digikey.jp/ja/products/detail/samsung-electro-m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
- C3: renamed from C7; Name GRM188R72A104KA35D -> GCJ188R91H124KA01D; Price 21 -> 36; URL https://www.digikey.jp/ja/products/detail/murata-electronics/GRM188R72A104KA35D/702549 -> https://www.digikey.jp/ja/products/detail/murata-electronics/GCJ188R91H124KA01D/13401917
- C4: value 0.1u -> 4.7u; Name GRM188R72A104KA35D -> GRM188R60G106ME47D; Price 21 -> 19; URL https://www.digikey.jp/ja/products/detail/murata-electronics/GRM188R72A104KA35D/702549 -> https://www.digikey.jp/ja/products/detail/murata-electronics/GRM188R60G106ME47D/702562
- D3: value PWM -> SW2; Name SMLEN3BC8TT86 -> SMLD12BN1WT86; Price 96 -> 48; URL https://www.digikey.jp/ja/products/detail/rohm-semiconductor/SMLEN3BC8TT86/15762415 -> https://www.digikey.jp/ja/products/detail/rohm-semiconductor/SMLD12BN1WT86/9826162
- D4: value MA -> SW1; Name SMLEN3BC8TT86 -> SMLD12BN1WT86; Price 96 -> 48; URL https://www.digikey.jp/ja/products/detail/rohm-semiconductor/SMLEN3BC8TT86/15762415 -> https://www.digikey.jp/ja/products/detail/rohm-semiconductor/SMLD12BN1WT86/9826162
- D5: value MB -> PWR; Name SMLEN3BC8TT86 -> SML-D12D8WT86; Price 96 -> 30; URL https://www.digikey.jp/ja/products/detail/rohm-semiconductor/SMLEN3BC8TT86/15762415 -> https://www.digikey.jp/ja/products/detail/rohm-semiconductor/SML-D12D8WT86/1641796
- D6: value PWR -> BATT; Name SML-E12P8WT86 -> SML-D12U8WT86; Price 41 -> 30; URL https://www.digikey.jp/ja/products/detail/rohm-semiconductor/SML-E12P8WT86/1641804 -> https://www.digikey.jp/ja/products/detail/rohm-semiconductor/SML-D12U8WT86/1641799
- R1: value 80 -> 420; Name ESR03EZPF82R0 -> ESR03EZPJ431; Price 24 -> 22; URL https://www.digikey.jp/ja/products/detail/rohm-semiconductor/ESR03EZPF82R0/4007286 -> https://www.digikey.jp/ja/products/detail/rohm-semiconductor/ESR03EZPJ431/4051257
- R10: value 20k -> 430; Name ESR03EZPF2002 -> ESR03EZPJ431; Price 24 -> 22; URL https://www.digikey.jp/ja/products/detail/rohm-semiconductor/ESR03EZPF2002/1983437 -> https://www.digikey.jp/ja/products/detail/rohm-semiconductor/ESR03EZPJ431/4051257
- R11: renamed from R16; value 500 -> 1.5k; Name ESR03EZPF4990 -> ESR03EZPJ152; Price 24 -> 22; URL https://www.digikey.jp/ja/products/detail/rohm-semiconductor/ESR03EZPF4990/21819734 -> https://www.digikey.jp/ja/products/detail/rohm-semiconductor/ESR03EZPJ152/1983456
- R2: value 80 -> 120; Name ESR03EZPF82R0 -> ESR03EZPJ121; Price 24 -> 22; URL https://www.digikey.jp/ja/products/detail/rohm-semiconductor/ESR03EZPF82R0/4007286 -> https://www.digikey.jp/ja/products/detail/rohm-semiconductor/ESR03EZPJ121/1983454
- R3: value 80 -> 100; Name ESR03EZPF82R0 -> ESR03EZPJ101; Price 24 -> 22; URL https://www.digikey.jp/ja/products/detail/rohm-semiconductor/ESR03EZPF82R0/4007286 -> https://www.digikey.jp/ja/products/detail/rohm-semiconductor/ESR03EZPJ101/1983452
- R4: value 80 -> 600; Name ESR03EZPF82R0 -> ESR03EZPF5900; Price 24 -> 22; URL https://www.digikey.jp/ja/products/detail/rohm-semiconductor/ESR03EZPF82R0/4007286 -> https://www.digikey.jp/ja/products/detail/rohm-semiconductor/ESR03EZPF5900/20506305
- R5: value 20k -> 300; Name ESR03EZPF2002 -> ESR03EZPJ301; Price 24 -> 22; URL https://www.digikey.jp/ja/products/detail/rohm-semiconductor/ESR03EZPF2002/1983437 -> https://www.digikey.jp/ja/products/detail/rohm-semiconductor/ESR03EZPJ301/1762729
- R6, R7: value 20k -> 330; Name ESR03EZPF2002 -> ESR03EZPJ331; Price 24 -> 22; URL https://www.digikey.jp/ja/products/detail/rohm-semiconductor/ESR03EZPF2002/1983437 -> https://www.digikey.jp/ja/products/detail/rohm-semiconductor/ESR03EZPJ331/1762730
- R8, R9: value 20k -> 80; Name ESR03EZPF2002 -> ESR03EZPJ820; Price 24 -> 22; URL https://www.digikey.jp/ja/products/detail/rohm-semiconductor/ESR03EZPF2002/1983437 -> https://www.digikey.jp/ja/products/detail/rohm-semiconductor/ESR03EZPJ820/4051294
- renumbered C10 to C5, C11 to C6, J1 to J5, U6 to U2
Connections:
- net MB is gone; now on an unnamed net: R6.2
- net at R3.1: now also U1.1; no longer R7.1
- net MCU/LED_R: now reaches R3.2
- net at R8.1: now also D3.1 (K); no longer R4.2
- net at R2.2: now also SW1.2 (B); no longer R6.1
- net at D4.1 (K): now also R9.1
- net at R1.2: now also SW1.5 (B)
- net at R4.1: now also U1.2
- net CAN/CAN_H: now reaches R2.1
- net CAN/CAN_H: now also J1.3 (Pin_3)
- net at R5.1: now also U1.3; no longer R1.1
- net at D5.1 (K): now also R10.1
- net at D4.2 (A): now also J3.1 (Pin_1)
- net +12V renamed +12VA
- net +12VA: no longer C4.1, D6.2 (A)
- net +24V renamed +BATT
- net +BATT: now also D6.2 (A)
- net DIR renamed +5VD
- net +5VD: now also C2.1, D1.1 (K), D2.2 (A), J2.4 (Pin_4), U3.3 (VI); no longer R10.1
- net GND renamed GNDD
- net GNDD: now also C4.2, R8.2, C2.2, H1.1, H2.1, J1.5 (Pin_5), J1.6 (Pin_6), J2.5 (Pin_5), JP1.3 (B), SW1.6 (C), SW2.1 (CM), U1.4, U1.5, U1.6, U3.1 (GND)
- net GNDPWR renamed GNDA
- net GNDA: now also H3.1, H4.1; no longer C4.2, R7.2, R8.2
- net MA renamed MCU/LED_G
- net PWM: no longer names the net of D3.2 (A)
- net PWM: now also R7.2, J4.1 (Pin_1); no longer R9.1
- new net: J3.2 (Pin_2), J4.2 (Pin_2), JP1.2 (C)
- new net: F1.2, J1.1 (Pin_1), J1.2 (Pin_2)
- new net: D1.2 (A), F1.1
- new net: D2.1 (K), R1.1
- new net +3.3VD: C4.1, JP1.1 (A), U3.2 (VO)
- new net CAN/CAN_L: J1.4 (Pin_4), SW1.3 (C)
- new net Driver/MA: J6.1 (Pin_1)
- new net Driver/MB: J6.2 (Pin_2)
- new net MCU/ENC_A/MISO: J2.3 (Pin_3)
- new net MCU/ENC_B/DATA: J2.2 (Pin_2)
- new net MCU/ID0: SW2.2 (D0)
- new net MCU/ID1: SW2.3 (D1)
- new net MCU/ID2: SW2.4 (D2)
- new net MCU/ID3: SW2.5 (D3)
- new net MCU/LED_B: R4.2
- new net MCU/SW1: R6.1
- new net MCU/SW2: R7.1
- new net MCU/X/SCK: J2.1 (Pin_1)
Other:
- added sheet CAN (MotorDriver_CAN.kicad_sch)
- added sheet Driver (MotorDriver_Driver.kicad_sch)
- added sheet Isolator (MotorDriver_Isolator.kicad_sch)
- added sheet MCU (MotorDriver_MCU.kicad_sch)
- added sheet USB-UART (MotorDriver_USB-UART.kicad_sch)
- note removed: "ロジック部"
- note removed: "電源・信号部"
- note removed: "駆動部"
- moved on the sheet: C1, C3, C5, C6, J5, R11, U2
