File: MotorDriver/MotorDriver_MCU.kicad_sch (KiCad schematic)
At the start: 15 parts, among them J7 SWD, SW3 RESET, U8 STM32F303K8Tx, Y1 Crystal_GND2

Commit message: Motor Driver ver2.1
Connections:
- net ENC_A/MISO: now also U8.18 (PA8); no longer U8.12 (PA6)
- net ENC_B/DATA: now also U8.19 (PA9); no longer U8.13 (PA7)
- net SW1: now also U8.12 (PA6); no longer U8.19 (PA9)
- net SW2: now also U8.13 (PA7); no longer U8.18 (PA8)
Other:
- note added: "PWM1: PB0: TIM3_CH3 PWM2: PB1: TIM3_CH4 ENC_A: PA8: TIM1_CH1 ENC_B: PA9: TIM1_CH2 VOUT: PA4: ADC2_IN1 LED_R: PA0: TIM2_CH1 LED_G: PA1: TIM2_CH2 LED_B: PA2: TIM2_CH3 UART2_TX: PB3 UART2_RX: PA15"
- note removed: "PWM1: PB0: TIM3_CH3 PWM2: PB1: TIM3_CH4 ENC_A: PA6: TIM3_CH1 ENC_B: PA7: TIM3_CH2 VOUT: PA4: ADC2_IN1 LED_R: PA0: TIM2_CH1 LED_G: PA1: TIM2_CH2 LED_B: PA2: TIM2_CH3 UART2_TX: PB3 UART2_RX: PA15"
Changed lines of the file:
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@@
 	(title_block
 		(title "MotorDriver / MCU")
-		(date "2025-07-11")
-		(rev "ver2.0")
+		(date "2025-08-19")
+		(rev "ver2.1")
 		(company "阿南高専ロボット研究部")
 	)
-	(text "PWM1: PB0: TIM3_CH3\nPWM2: PB1: TIM3_CH4\n\nENC_A: PA6: TIM3_CH1\nENC_B: PA7: TIM3_CH2\n\nVOUT: PA4: ADC2_IN1\n\nLED_R: PA0: TIM2_CH1\nLED_G: PA1: TIM2_CH2\nLED_B: PA2: TIM2_CH3\n\nUART2_TX: PB3\nUART2_RX: PA15"
+	(text "PWM1: PB0: TIM3_CH3\nPWM2: PB1: TIM3_CH4\n\nENC_A: PA8: TIM1_CH1\nENC_B: PA9: TIM1_CH2\n\nVOUT: PA4: ADC2_IN1\n\nLED_R: PA0: TIM2_CH1\nLED_G: PA1: TIM2_CH2\nLED_B: PA2: TIM2_CH3\n\nUART2_TX: PB3\nUART2_RX: PA15"
 		(exclude_from_sim no)
 		(at 200.025 92.71 0)
@@
 	(hierarchical_label "ENC_A{slash}MISO"
 		(shape input)
-		(at 161.29 97.155 0)
+		(at 161.29 102.235 0)
+		(effects
+			(font
+				(size 1.27 1.27)
+			)
+			(justify left)
+		)
+	)
+	(hierarchical_label "SW2"
+		(shape input)
+		(at 161.29 99.695 0)
 		(effects
 			(font
@@
 		)
 	)
-	(hierarchical_label "ENC_B{slash}DATA"
-		(shape input)
-		(at 161.29 99.695 0)
-		(effects
-			(font
-				(size 1.27 1.27)
-			)
-			(justify left)
-		)
-	)
 	(hierarchical_label "UART2_RX"
 		(shape input)
@@
 		)
 	)
-	(hierarchical_label "SW2"
-		(shape input)
-		(at 161.29 102.235 0)
+	(hierarchical_label "SW1"
+		(shape input)
+		(at 161.29 97.155 0)
 		(effects
 			(font
@@
 		)
 	)
-	(hierarchical_label "SW1"
+	(hierarchical_label "ENC_B{slash}DATA"
 		(shape input)
 		(at 161.29 104.775 0)
