File: ConverterBoard/ConverterBoard.kicad_sch (KiCad schematic)
At the start: 51 parts, among them J1 PWR_IN, J2 PWR_OUT1, J3 PWR_OUT2, J4 PWR_OUT3, U1 RT6285, U2 RT6285, U3 RT6285

Commit message: Converter Board ver1.1
Parts:
- D1, D2, D3: footprint Diode_SMD:D_SMA -> Diode_SMD:D_SMC
- U1, U2, U3: footprint Package_SO:SOIC-8-1EP_3.9x4.9mm_P1.27mm_EP2.29x3mm_ThermalVias -> Anan-Robo_Footprint_Library:SOIC-8-1EP_3.9x4.9mm_P1.27mm_EP2.29x3mm_Handsoldering
Other:
- note added: "20kgサーボモーター用など"
- note removed: "20kgサーボモーター用"
Changed lines of the file:
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@@
 	(title_block
 		(title "Converter Board")
-		(date "2025-05-31")
-		(rev "ver1.0")
+		(date "2025-06-17")
+		(rev "ver1.1")
 		(company "阿南高専ロボット研究部")
 	)
-	(text "20kgサーボモーター用"
+	(text "20kgサーボモーター用など"
 		(exclude_from_sim no)
 		(at 207.01 102.87 0)
@@
 			)
 		)
-		(property "Footprint" "Diode_SMD:D_SMA"
+		(property "Footprint" "Diode_SMD:D_SMC"
 			(at 147.32 72.39 0)
 			(effects
@@
 			)
 		)
-		(property "Footprint" "Package_SO:SOIC-8-1EP_3.9x4.9mm_P1.27mm_EP2.29x3mm_ThermalVias"
+		(property "Footprint" "Anan-Robo_Footprint_Library:SOIC-8-1EP_3.9x4.9mm_P1.27mm_EP2.29x3mm_Handsoldering"
 			(at 129.54 88.9 0)
 			(effects
@@
 			)
 		)
-		(property "Footprint" "Package_SO:SOIC-8-1EP_3.9x4.9mm_P1.27mm_EP2.29x3mm_ThermalVias"
+		(property "Footprint" "Anan-Robo_Footprint_Library:SOIC-8-1EP_3.9x4.9mm_P1.27mm_EP2.29x3mm_Handsoldering"
 			(at 129.54 125.73 0)
 			(effects
@@
 			)
 		)
-		(property "Footprint" "Diode_SMD:D_SMA"
+		(property "Footprint" "Diode_SMD:D_SMC"
 			(at 147.32 146.05 0)
 			(effects
@@
 			)
 		)
-		(property "Footprint" "Diode_SMD:D_SMA"
+		(property "Footprint" "Diode_SMD:D_SMC"
 			(at 147.32 109.22 0)
 			(effects
@@
 			)
 		)
-		(property "Footprint" "Package_SO:SOIC-8-1EP_3.9x4.9mm_P1.27mm_EP2.29x3mm_ThermalVias"
+		(property "Footprint" "Anan-Robo_Footprint_Library:SOIC-8-1EP_3.9x4.9mm_P1.27mm_EP2.29x3mm_Handsoldering"
 			(at 129.54 52.07 0)
 			(effects

Commit message: Converter Board ver1.2
Parts:
- added D4: BATT, LED_SMD:LED_0603_1608Metric, symbol Device:LED
- added D5: 5V, LED_SMD:LED_0603_1608Metric, symbol Device:LED
- added D6: 6.5V, LED_SMD:LED_0603_1608Metric, symbol Device:LED
- added D7: 12V, LED_SMD:LED_0603_1608Metric, symbol Device:LED
- added R10: 500, Resistor_SMD:R_0603_1608Metric, symbol Device:R
- added R7: 1.5k, Resistor_SMD:R_0603_1608Metric, symbol Device:R
- added R8: 240, Resistor_SMD:R_0603_1608Metric, symbol Device:R
- added R9: 390, Resistor_SMD:R_0603_1608Metric, symbol Device:R
- C7, C8, C9: Name GRM1885C1H103JA01D -> GCM1885C1H103JA16D; Price 19 -> 26; URL https://www.digikey.jp/ja/products/detail/murata-electronics/GRM1885C1H103JA01D/4421555 -> https://www.digikey.jp/ja/products/detail/murata-electronics/GCM1885C1H103JA16D/13402328
- L3: value 33u -> 22u; Name NR10050T330M -> NR10050T220M; URL https://www.digikey.jp/ja/products/detail/taiyo-yuden/NR10050T330M/1171799 -> https://www.digikey.jp/ja/products/detail/taiyo-yuden/NR10050T220M/1007973
- R6: value 11.3k -> 18k; Name RG1608P-1132-B-T5 -> RN73H1JTTD1802B25; Price 18 -> 32; URL https://www.digikey.jp/ja/products/detail/susumu/RG1608P-11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 -> https://www.digikey.jp/ja/products/detail/koa-speer-electro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
Connections:
- net +5VA: now also D5.2 (A)
- net +6.5VA: now also D6.2 (A)
- net +BATT: now also D4.2 (A)
- net GND: now also R10.2, R7.2, R8.2, R9.2
- net +12VA renamed +8VA
- net +8VA: now also D7.2 (A)
- new net: D6.1 (K), R9.1
- new net: D5.1 (K), R8.1
- new net: D4.1 (K), R7.1
- new net: D7.1 (K), R10.1
Other:
- note added: "20kgサーボモーター用"
- note added: "60kgサーボモーター用"
- note removed: "100kgサーボモーター、バキュームポンプ用など"
- note removed: "20kgサーボモーター用など"
- moved on the sheet: C1, C10, C11, C12, C13, C14, C15, C16, C17, C18, C19, C2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
