File: XT30Hub/XT30Hub.kicad_pcb (KiCad board)
At the start: 2 copper layers, 65.5 x 26.9 mm, 15 parts, among them J1 Conn_01x02, J2 Conn_01x02, J3 Conn_01x02, J4 Conn_01x02, J5 Conn_01x02, J6 Conn_01x02

Commit message: [XT30Hub] : 裏面の枠線の太さを修正
Other:
- board text added: "ver 1.0: 2025-04-07"
- board text removed: "ver 1.0: 2025-04-01"
Changed lines of the file:
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@@
 		(end 134.07 113)
 		(stroke
-			(width 0.1)
-			(type default)
+			(width 0.12)
+			(type solid)
 		)
 		(layer "B.SilkS")
@@
 		(end 175 97.5)
 		(stroke
-			(width 0.1)
-			(type default)
+			(width 0.12)
+			(type solid)
 		)
 		(layer "B.SilkS")
@@
 		(end 183 113)
 		(stroke
-			(width 0.1)
-			(type default)
+			(width 0.12)
+			(type solid)
 		)
 		(layer "B.SilkS")
@@
 		(end 162 97.5)
 		(stroke
-			(width 0.1)
-			(type default)
+			(width 0.12)
+			(type solid)
 		)
 		(layer "B.SilkS")
@@
 		(end 134.07 97.5)
 		(stroke
-			(width 0.1)
-			(type default)
+			(width 0.12)
+			(type solid)
 		)
 		(layer "B.SilkS")
@@
 		)
 	)
-	(gr_text "ver 1.0: 2025-04-01"
+	(gr_text "ver 1.0: 2025-04-07"
 		(at 128 96 180)
 		(layer "B.SilkS")
@@
 			(justify left mirror)
 		)
-		(render_cache "ver 1.0: 2025-04-01" 180
+		(render_cache "ver 1.0: 2025-04-07" 180
 			(polygon
 				(pts
@@
 			(polygon
 				(pts
-					(xy 143.323674 95.762625) (xy 143.54911 95.762625) (xy 143.54911 96.396557) (xy 143.396092 96.231205)
-					(xy 143.300409 96.330978) (xy 143.550453 96.604225) (xy 143.744443 96.604225) (xy 143.744443 95.762625)
-					(xy 143.971222 95.762625) (xy 143.971222 95.585) (xy 143.323674 95.585)
-				)
-			)
+					(xy 143.713058 96.426599) (xy 143.288136 96.426599) (xy 143.288136 96.604225) (xy 143.932998 96.604225)
+					(xy 143.932998 96.462137) (xy 143.58599 95.585) (xy 143.38101 95.585)
+				)
+			)

Commit message: [XT30Hub] : 発注前に最終調整
Other:
- board text added: "ver 1.0: 2025-04-12"
- board text removed: "ver 1.0: 2025-04-07"
Changed lines of the file:
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@@
 		)
 	)
-	(gr_text "ver 1.0: 2025-04-07"
+	(gr_text "ver 1.0: 2025-04-12"
 		(at 128 96 180)
 		(layer "B.SilkS")
@@
 			(justify left mirror)
 		)
-		(render_cache "ver 1.0: 2025-04-07" 180
+		(render_cache "ver 1.0: 2025-04-12" 180
 			(polygon
 				(pts
@@
 			(polygon
 				(pts
-					(xy 142.792763 95.98189) (xy 142.812294 95.992057) (xy 142.829998 96.00986) (xy 142.847519 96.044967)
-					(xy 142.853934 96.093269) (xy 142.847542 96.141611) (xy 142.829998 96.177227) (xy 142.81224 96.195487)
-					(xy 142.792711 96.205867) (xy 142.770586 96.209345) (xy 142.748457 96.205869) (xy 142.728907 96.195489)
-					(xy 142.711113 96.177227) (xy 142.693615 96.141616) (xy 142.687238 96.093269) (xy 142.693864 96.045242)
-					(xy 142.711845 96.011264) (xy 142.729244 95.992605) (xy 142.748539 95.982023) (xy 142.770586 95.978475)
-				)
-			)
-			(polygon
-				(pts
-					(xy 142.829915 95.569954) (xy 142.881429 95.581534) (xy 142.926352 95.60002) (xy 142.967325 95.626061)
-					(xy 143.003642 95.659095) (xy 143.03565 95.699794) (xy 143.071474 95.767258) (xy 143.099318 95.852676)
-					(xy 143.117706 95.959874) (xy 143.124433 96.093269) (xy 143.117676 96.228178) (xy 143.099234 96.336232)
-					(xy 143.071366 96.421998) (xy 143.035589 96.489431) (xy 142.996562 96.537654) (xy 142.951554 96.574491)
-					(xy 142.899833 96.601044) (xy 142.840099 96.617546) (xy 142.770586 96.623337) (xy 142.716649 96.619659)
-					(xy 142.666755 96.608894) (xy 142.620254 96.591219) (xy 142.577759 96.566068) (xy 142.539638 96.532465)
-					(xy 142.505521 96.489431) (xy 142.469601 96.42063) (xy 142.441758 96.334199) (xy 142.423426 96.226483)
-					(xy 142.416806 96.094612) (xy 142.624406 96.094612) (xy 142.62949 96.219921) (xy 142.642344 96.304848)
-					(xy 142.659944 96.359677) (xy 142.681586 96.398069) (xy 142.706824 96.423284) (xy 142.736018 96.437984)
-					(xy 142.770586 96.443025) (xy 142.805859 96.437947) (xy 142.835493 96.423182) (xy 142.860953 96.397954)
-					(xy 142.882632 96.359677) (xy 142.900201 96.304851) (xy 142.913033 96.219924) (xy 142.918108 96.094612)
-					(xy 142.913023 95.968363) (xy 142.900181 95.883056) (xy 142.882632 95.828204) (xy 142.861028 95.790641)
-					(xy 142.835606 95.765803) (xy 142.805948 95.751223) (xy 142.770586 95.7462) (xy 142.735929 95.751186)
-					(xy 142.706712 95.765703) (xy 142.681512 95.790528) (xy 142.659944 95.828204) (xy 142.642364 95.883059)
-					(xy 142.6295 95.968365) (xy 142.624406 96.094612) (xy 142.416806 96.094612) (xy 142.416739 96.093269)
-					(xy 142.423509 95.958287) (xy 142.441965 95.850484) (xy 142.469815 95.765197) (xy 142.505521 95.698389)
-					(xy 142.537409 95.658524) (xy 142.573506 95.625937) (xy 142.614148 95.60002) (xy 142.658652 95.581596)
-					(xy 142.710344 95.569987) (xy 142.770586 95.565887)
-				)
-			)
-			(polygon
-				(pts
-					(xy 143.713058 96.426599) (xy 143.288136 96.426599) (xy 143.288136 96.604225) (xy 143.932998 96.604225)
-					(xy 143.932998 96.462137) (xy 143.58599 95.585) (xy 143.38101 95.585)
-				)
-			)
+					(xy 142.47957 95.762625) (xy 142.705006 95.762625) (xy 142.705006 96.396557) (xy 142.551988 96.231205)
+					(xy 142.456306 96.330978) (xy 142.70635 96.604225) (xy 142.90034 96.604225) (xy 142.90034 95.762625)
+					(xy 143.127119 95.762625) (xy 143.127119 95.585) (xy 142.47957 95.585)
+				)
+			)
+			(polygon
+				(pts
+					(xy 143.274459 95.732583) (xy 143.278479 95.754541) (xy 143.290884 95.774898) (xy 143.383757 95.873267)
+					(xy 143.503986 96.002411) (xy 143.572313 96.076844) (xy 143.61878 96.128745) (xy 143.662438 96.183394)
+					(xy 143.692541 96.232609) (xy 143.709458 96.279462) (xy 143.715744 96.324139) (xy 143.710792 96.366008)
+					(xy 143.696827 96.399762) (xy 143.67404 96.427271) (xy 143.644152 96.447399) (xy 143.606012 96.460225)
+					(xy 143.557292 96.464884) (xy 143.498455 96.459587) (xy 143.435659 96.443025) (xy 143.367332 96.417013)
+					(xy 143.296318 96.380132) (xy 143.296318 96.568688) (xy 143.374171 96.593967) (xy 143.438407 96.609659)
+					(xy 143.508948 96.620001) (xy 143.575061 96.623337) (xy 143.647475 96.618805) (xy 143.714401 96.605568)
+					(xy 143.776163 96.582017) (xy 143.827791 96.548171) (xy 143.866533 96.508777) (xy 143.895385 96.461465)
+					(xy 143.912984 96.407047) (xy 143.919321 96.33916) (xy 143.914609 96.284893) (xy 143.900209 96.229862)
+					(xy 143.87099 96.171299) (xy 143.830539 96.112381) (xy 143.760136 96.034467) (xy 143.632397 95.903309)
+					(xy 143.553872 95.829548) (xy 143.506734 95.79401) (xy 143.471196 95.762625) (xy 143.922069 95.762625)
+					(xy 143.922069 95.585) (xy 143.274459 95.585)
+				)
+			)

Commit message: XT30 Hub ver1.1
Parts:
- moved REF** 3.00 mm to (168.5, 95.2)
- moved H1 0.25 mm to (124.0, 95.0)
- moved H3 0.25 mm to (182.6, 95.0)
- moved H4 0.25 mm to (124.0, 115.5)
- moved H6 0.25 mm to (182.6, 115.5)
Routing:
- removed copper zone on B.Cu, net +BATT
- removed copper zone on B.Cu, net GND
Other:
- board size 65.5 x 26.9 mm -> 65.5 x 27.4 mm
- board text added: "ver 1.1: 2025-09-10"
- board text added: "ver1.1 by yuta"
- board text removed: "ver 1.0: 2025-04-12"
- board text removed: "ver1.0 by yuta"
